File: hw/Telemetry.sch (KiCad schematic (older format))
At the start: 28 parts

Commit message: Removed inverters and added expansion port
Parts:
- removed Q? (x4): BSS138, Package_TO_SOT_SMD:SOT-23, symbol Transistor_FET:BSS138
- removed R? (x7): 10k, symbol Device:R
- removed R?: 100k, symbol Device:R
- removed R?: 100, symbol Device:R
- removed R?: 10, symbol Device:R
- added J?: EXP, symbol Connector_Generic:Conn_01x06
- added SW?: SW_Push, symbol Switch:SW_Push
Connections:
- net labels removed: S.portRx, S.portTX, SbusRx, SbusTx
- wire segments 124 -> 111

Commit message: Updated pin assignments and preliminary timer2 setup
Signed-off-by: findersee <aki.kuusela@findersee.fi>
Parts:
- gave numbers to parts that had none: 16
Connections:
- net labels added: HC_OUT1, OUT1, OUT2, OUT3, OUT4, OUT5, OUT6, SERVO_OUT1, SERVO_OUT2, SERVO_OUT3, SERVO_OUT4, SPI_CS, SPI_MISO, SPI_MOSI, SPI_SCK
- wire segments 111 -> 121

Commit message: Connections updates
Parts:
- removed D101: D_Schottky, symbol Device:D_Schottky
- removed J101: EXP, symbol Connector_Generic:Conn_01x06
- added J101: VS1053 EXP, Pin_Headers:Pin_Header_Straight_1x10, symbol Connector_Generic:Conn_01x10
- added J106: UART_EXP, Pin_Headers:Pin_Header_Straight_1x04, symbol Connector_Generic:Conn_01x04
- added JP101: Jumper_NC_Small, Pin_Headers:Pin_Header_Angled_1x02, symbol Device:Jumper_NC_Small
- C101, C102, C103, C104, C105: footprint (none) -> Capacitors_SMD:C_0603_HandSoldering
- J102: footprint (none) -> Pin_Headers:Pin_Header_Straight_1x02
- J103, J104: footprint (none) -> Pin_Headers:Pin_Header_Angled_2x03
- J105: footprint (none) -> Connect:USB_Micro-B
- R101, R102, SW101: footprint (none) -> Resistors_SMD:R_0603_HandSoldering
- U101: footprint (none) -> Housings_QFP:LQFP-48_7x7mm_Pitch0.5mm
Connections:
- net labels added: BAT_VOLTAGE, DREQ, UART_RX, UART_TX, XCS, XDCS, XRESET
- wire segments 121 -> 137

Commit message: Layout started, schematic modified for easier layout
Parts:
- JP101: footprint Pin_Headers:Pin_Header_Angled_1x02 -> Pin_Headers:Pin_Header_Straight_1x02
- SW101: footprint Resistors_SMD:R_0603_HandSoldering -> digikey-footprints:Switch_Tactile_SMD_B3U-1000P
- X101: footprint Oscillator:Oscillator_SMD_TXC_7C-4Pin_5.0x3.2mm -> PCBDecals:IQXO-791
Connections:
- net labels added: HC_OUT2
Changed lines of the file:
@@
 Wire Wire Line
 	4850 6150 4850 6100
-$Comp
-L Oscillator:TXC-7C X101
-U 1 1 5CE21410
-P 3900 2000
-F 0 "X101" H 4000 2250 50  0000 L CNN
-F 1 "TXC-7C" H 4000 1750 50  0000 L CNN
-F 2 "Oscillator:Oscillator_SMD_TXC_7C-4Pin_5.0x3.2mm" H 4600 1650 50  0001 C CNN
-F 3 "http://www.txccorp.com/download/products/osc/7C_o.pdf" H 3800 2000 50  0001 C CNN
-	1    3900 2000
-	1    0    0    -1
-$EndComp
 Wire Wire Line
 	4850 2000 4200 2000
@@
 F 0 "SW101" H 4400 1135 50  0000 C CNN
 F 1 "SW_Push" H 4400 1044 50  0000 C CNN
-F 2 "Resistors_SMD:R_0603_HandSoldering" H 4400 1050 50  0001 C CNN
+F 2 "digikey-footprints:Switch_Tactile_SMD_B3U-1000P" H 4400 1050 50  0001 C CNN
 F 3 "" H 4400 1050 50  0001 C CNN
 	1    4400 850
@@
 Wire Wire Line
 	6050 2700 6150 2700
-Text GLabel 6150 3600 2    50   Output ~ 0
+Text GLabel 6150 2700 2    50   Output ~ 0
 OUT2
 Wire Wire Line
@@
 HC_OUT1
 Text GLabel 6150 3400 2    50   Output ~ 0
-HC_OUT1
+HC_OUT2
 Text GLabel 6150 2300 2    50   Output ~ 0
 OUT1
@@
 Wire Wire Line
 	6150 3600 6050 3600
-Text GLabel 6150 2700 2    50   Output ~ 0
+Text GLabel 6150 2900 2    50   Output ~ 0
 OUT3
+Text GLabel 6150 3600 2    50   Output ~ 0
+OUT4
 Text GLabel 6150 2800 2    50   Output ~ 0
-OUT4
-Text GLabel 6150 2900 2    50   Output ~ 0
 OUT5
 Text GLabel 6150 3100 2    50   Output ~ 0
@@
 F 0 "JP101" V 9846 1403 50  0000 R CNN
 F 1 "Jumper_NC_Small" V 9755 1403 50  0000 R CNN
-F 2 "Pin_Headers:Pin_Header_Angled_1x02" H 9800 1450 50  0001 C CNN
+F 2 "Pin_Headers:Pin_Header_Straight_1x02" H 9800 1450 50  0001 C CNN
 F 3 "~" H 9800 1450 50  0001 C CNN
 	1    9800 1450
@@
 Wire Wire Line
 	4100 6150 4850 6150
+$Comp
+L Oscillator:TXC-7C X101
+U 1 1 5CE6962F
+P 3900 2000
+F 0 "X101" H 4241 2046 50  0000 L CNN
+F 1 "TXC-7C" H 4241 1955 50  0000 L CNN
+F 2 "PCBDecals:IQXO-791" H 4600 1650 50  0001 C CNN
+F 3 "http://www.txccorp.com/download/products/osc/7C_o.pdf" H 3800 2000 50  0001 C CNN
+	1    3900 2000
+	1    0    0    -1
+$EndComp
 $EndSCHEMATC

Commit message: Continued layout Setup USB device CDC
Connections:
- no-connect marks 0 -> 5
Changed lines of the file:
@@
 	1    0    0    -1
 $EndComp
+NoConn ~ 4850 2200
+NoConn ~ 6050 4000
+NoConn ~ 6050 4400
+NoConn ~ 6050 4500
+NoConn ~ 6050 4600
 $EndSCHEMATC

Commit message: Layout improvements
Signed-off-by: findersee <aki.kuusela@findersee.fi>
Parts:
- J102: footprint Pin_Headers:Pin_Header_Straight_1x02 -> Pin_Headers:Pin_Header_Straight_1x02_Pitch1.00mm
- SW101: footprint digikey-footprints:Switch_Tactile_SMD_B3U-1000P -> Pin_Headers:Pin_Header_Straight_1x02_Pitch1.27mm
Connections:
- net labels added: VBUS
Changed lines of the file:
@@
 F 0 "J102" H 2920 875 50  0000 C CNN
 F 1 "BOOT0" H 2920 966 50  0000 C CNN
-F 2 "Pin_Headers:Pin_Header_Straight_1x02" H 3000 1200 50  0001 C CNN
+F 2 "Pin_Headers:Pin_Header_Straight_1x02_Pitch1.00mm" H 3000 1200 50  0001 C CNN
 F 3 "~" H 3000 1200 50  0001 C CNN
 	1    3000 1200
@@
 $EndComp
 Wire Wire Line
-	4100 6350 4400 6350
-Wire Wire Line
-	4100 6450 4400 6450
-Text Label 4400 6450 0    50   ~ 0
+	4100 6350 4200 6350
+Wire Wire Line
+	4100 6450 4200 6450
+Text Label 4200 6450 0    50   ~ 0
 USB_D-
-Text Label 4400 6350 0    50   ~ 0
+Text Label 4200 6350 0    50   ~ 0
 USB_D+
 $Comp
@@
 	3800 6800 3800 6750
 Connection ~ 3800 6800
-Wire Wire Line
-	4850 6150 4850 6100
 Wire Wire Line
 	4850 2000 4200 2000
@@
 F 0 "SW101" H 4400 1135 50  0000 C CNN
 F 1 "SW_Push" H 4400 1044 50  0000 C CNN
-F 2 "digikey-footprints:Switch_Tactile_SMD_B3U-1000P" H 4400 1050 50  0001 C CNN
+F 2 "Pin_Headers:Pin_Header_Straight_1x02_Pitch1.27mm" H 4400 1050 50  0001 C CNN
 F 3 "" H 4400 1050 50  0001 C CNN
 	1    4400 850
@@
 Text Label 6750 3500 0    50   ~ 0
 DREQ
-$Comp
-L power:VCC #PWR0112
-U 1 1 5CED9BFF
-P 4850 6100
-F 0 "#PWR0112" H 4850 5950 50  0001 C CNN
-F 1 "VCC" H 4867 6273 50  0000 C CNN
-F 2 "" H 4850 6100 50  0001 C CNN
-F 3 "" H 4850 6100 50  0001 C CNN
-	1    4850 6100
-	1    0    0    -1
-$EndComp
-Wire Wire Line
-	4100 6150 4850 6150
+Wire Wire Line
+	4100 6150 4200 6150
 $Comp
 L Oscillator:TXC-7C X101
@@
 NoConn ~ 6050 4500
 NoConn ~ 6050 4600
+Wire Wire Line
+	4200 6150 4200 6100
+$Comp
+L power:VBUS #PWR0112
+U 1 1 5CEEB052
+P 4200 6100
+F 0 "#PWR0112" H 4200 5950 50  0001 C CNN
+F 1 "VBUS" H 4215 6273 50  0000 C CNN
+F 2 "" H 4200 6100 50  0001 C CNN
+F 3 "" H 4200 6100 50  0001 C CNN
+	1    4200 6100
+	1    0    0    -1
+$EndComp
 $EndSCHEMATC

Commit message: Added DAC initialization Added 32Mbit SPI FLASH memory Removed SPI expansion port
Parts:
- removed J101: VS1053 EXP, Pin_Headers:Pin_Header_Straight_1x10, symbol Connector_Generic:Conn_01x10
- added D?: LED, symbol Device:LED
- added U?: IS25LP032D, symbol Misc:IS25LP032D
- J102: footprint Pin_Headers:Pin_Header_Straight_1x02_Pitch1.00mm -> Pin_Headers:Pin_Header_Straight_1x02_Pitch1.27mm
Connections:
- net labels added: COOLING_TEMP, DAC_OUT, WP
- net labels removed: DREQ, XCS, XDCS, XRESET
- wire segments 137 -> 140
- no-connect marks 5 -> 6
Other:
- note added: "ERROR LED"

Commit message: Fixed crash problems
Parts:
- added C106: 100n, Capacitors_SMD:C_0603_HandSoldering, symbol Device:C_Small
- added R103: 470R, Resistors_SMD:R_0603_HandSoldering, symbol Device:R
- D101: renamed from D?; footprint (none) -> LEDs:LED_0603_HandSoldering
- U102: renamed from U?; footprint (none) -> digikey-footprints:SOIC-8_W3.9mm
Connections:
- wire segments 140 -> 144
Changed lines of the file:
@@
 	7950 1200 9450 1200
 $Comp
-L Misc:IS25LP032D U?
+L Misc:IS25LP032D U102
 U 1 1 5CEB0F5A
 P 9900 1400
-F 0 "U?" H 9900 1975 50  0000 C CNN
+F 0 "U102" H 9900 1975 50  0000 C CNN
 F 1 "IS25LP032D" H 9900 1884 50  0000 C CNN
-F 2 "" H 9800 1250 50  0001 C CNN
+F 2 "digikey-footprints:SOIC-8_W3.9mm" H 9800 1250 50  0001 C CNN
 F 3 "" H 9800 1250 50  0001 C CNN
 	1    9900 1400
@@
 	6050 1500 9450 1500
 $Comp
-L power:+3V3 #PWR?
+L power:+3V3 #PWR0101
 U 1 1 5CEF7FBB
-P 9400 1000
-F 0 "#PWR?" H 9400 850 50  0001 C CNN
-F 1 "+3V3" H 9415 1173 50  0000 C CNN
-F 2 "" H 9400 1000 50  0001 C CNN
-F 3 "" H 9400 1000 50  0001 C CNN
-	1    9400 1000
+P 9400 750
+F 0 "#PWR0101" H 9400 600 50  0001 C CNN
+F 1 "+3V3" H 9415 923 50  0000 C CNN
+F 2 "" H 9400 750 50  0001 C CNN
+F 3 "" H 9400 750 50  0001 C CNN
+	1    9400 750
 	1    0    0    -1
 $EndComp
@@
 	9450 1050 9400 1050
 Wire Wire Line
-	9400 1050 9400 1000
+	9400 1050 9400 750
 Wire Wire Line
 	6050 2000 8300 2000
@@
 NoConn ~ 6050 3200
 $Comp
-L Device:LED D?
+L Device:LED D101
 U 1 1 5CF14422
 P 7100 4400
-F 0 "D?" H 7091 4616 50  0000 C CNN
+F 0 "D101" H 7091 4616 50  0000 C CNN
 F 1 "LED" H 7091 4525 50  0000 C CNN
-F 2 "" H 7100 4400 50  0001 C CNN
+F 2 "LEDs:LED_0603_HandSoldering" H 7100 4400 50  0001 C CNN
 F 3 "~" H 7100 4400 50  0001 C CNN
 	1    7100 4400
@@
 $EndComp
 $Comp
-L power:+3V3 #PWR?
+L power:+3V3 #PWR0125
 U 1 1 5CF145CC
 P 7450 4300
-F 0 "#PWR?" H 7450 4150 50  0001 C CNN
+F 0 "#PWR0125" H 7450 4150 50  0001 C CNN
 F 1 "+3V3" H 7465 4473 50  0000 C CNN
 F 2 "" H 7450 4300 50  0001 C CNN
@@
 Wire Wire Line
 	7450 4400 7250 4400
-Wire Wire Line
-	6050 4400 6950 4400
 $Comp
 L Misc:STM32F303CBx U101
@@
 Text Notes 7200 4500 0    50   ~ 0
 ERROR LED
+$Comp
+L Device:R R103
+U 1 1 5CF2EC11
+P 6600 4400
+F 0 "R103" V 6500 4400 50  0000 C CNN
+F 1 "470R" V 6600 4400 50  0000 C CNN
+F 2 "Resistors_SMD:R_0603_HandSoldering" V 6530 4400 50  0001 C CNN
+F 3 "~" H 6600 4400 50  0001 C CNN
+	1    6600 4400
+	0    1    1    0
+$EndComp
+Wire Wire Line
+	6950 4400 6750 4400
+Wire Wire Line
+	6050 4400 6450 4400
+$Comp
+L Device:C_Small C106
+U 1 1 5CF3E241
+P 10400 1400
+F 0 "C106" H 10492 1446 50  0000 L CNN
+F 1 "100n" H 10492 1355 50  0000 L CNN
+F 2 "Capacitors_SMD:C_0603_HandSoldering" H 10400 1400 50  0001 C CNN
+F 3 "~" H 10400 1400 50  0001 C CNN
+	1    10400 1400
+	1    0    0    -1
+$EndComp
+Wire Wire Line
+	10400 1300 10400 750
+Wire Wire Line
+	10400 750  9400 750
+Connection ~ 9400 750
+Wire Wire Line
+	10400 1500 10400 1750
+Connection ~ 10400 1750
 $EndSCHEMATC
