File: hw/Telemetry.sch (KiCad schematic (older format))
At the start: 20 parts, among them J102 BOOT0, J103 SPORT, J104 SBUS, J105 USB_B_Micro, J106 UART_EXP, SW101 SW_Push, U101 STM32F303CBx, U102 IS25LP032D, X101 TXC-7C

Commit message: Added DAC output connector to the design
Parts:
- added C107: 10u, Capacitors_SMD:C_0603_HandSoldering, symbol Device:C_Small
- added C108: 10p, Capacitors_SMD:C_0603_HandSoldering, symbol Device:C_Small
- added J101: AUDIO, Pin_Headers:Pin_Header_Straight_1x02_Pitch2.54mm, symbol Connector_Generic:Conn_01x02
- added MH101, MH102, MH103, MH104: MountingHole, Mounting_Holes:MountingHole_3.2mm_M3_DIN965, symbol Mechanical:MountingHole
Connections:
- net labels removed: DAC_OUT
- wire segments 144 -> 153
Changed lines of the file:
@@
 Wire Wire Line
 	8450 3100 9000 3100
-Wire Wire Line
-	6050 1400 6200 1400
-Wire Wire Line
-	6050 1600 8050 1600
 $Comp
 L power:GND #PWR0104
@@
 	7950 1200 7950 1800
 Wire Wire Line
-	7950 1800 6050 1800
-Text GLabel 6200 1400 2    50   Output ~ 0
-DAC_OUT
-Wire Wire Line
 	6050 2400 8300 2400
 Wire Wire Line
@@
 Wire Wire Line
 	7950 1200 9450 1200
-$Comp
-L Misc:IS25LP032D U102
-U 1 1 5CEB0F5A
-P 9900 1400
-F 0 "U102" H 9900 1975 50  0000 C CNN
-F 1 "IS25LP032D" H 9900 1884 50  0000 C CNN
-F 2 "digikey-footprints:SOIC-8_W3.9mm" H 9800 1250 50  0001 C CNN
-F 3 "" H 9800 1250 50  0001 C CNN
-	1    9900 1400
-	1    0    0    -1
-$EndComp
 Wire Wire Line
 	10350 1750 10400 1750
 Wire Wire Line
 	10400 1750 10400 1800
-Wire Wire Line
-	9450 1300 8050 1300
-Wire Wire Line
-	8050 1300 8050 1600
-Wire Wire Line
-	8150 1400 8150 1700
-Wire Wire Line
-	6050 1700 8150 1700
-Wire Wire Line
-	8150 1400 9450 1400
-Wire Wire Line
-	6050 1500 9450 1500
 $Comp
 L power:+3V3 #PWR0101
@@
 Wire Wire Line
 	9400 1050 9400 750
-Wire Wire Line
-	6050 2000 8300 2000
-Wire Wire Line
-	8300 2000 8300 1750
 Text Label 8550 1750 0    50   ~ 0
 WP
-Wire Wire Line
-	9450 1750 8300 1750
 NoConn ~ 9450 1650
 NoConn ~ 6050 3500
@@
 	10400 1500 10400 1750
 Connection ~ 10400 1750
+$Comp
+L Device:C_Small C107
+U 1 1 5CE9FBD8
+P 7300 1400
+F 0 "C107" V 7071 1400 50  0000 C CNN
+F 1 "10u" V 7162 1400 50  0000 C CNN
+F 2 "Capacitors_SMD:C_0603_HandSoldering" H 7300 1400 50  0001 C CNN
+F 3 "~" H 7300 1400 50  0001 C CNN
+	1    7300 1400
+	0    1    1    0
+$EndComp
+Wire Wire Line
+	7450 1400 7400 1400
+Wire Wire Line
+	6050 1400 7200 1400
+$Comp
+L Misc:IS25LP032D U102
+U 1 1 5CEB0F5A
+P 9900 1400
+F 0 "U102" H 9900 1975 50  0000 C CNN
+F 1 "IS25LP032D" H 9900 1884 50  0000 C CNN
+F 2 "digikey-footprints:SOIC-8_W3.9mm" H 9800 1250 50  0001 C CNN
+F 3 "" H 9800 1250 50  0001 C CNN
+	1    9900 1400
+	1    0    0    -1
+$EndComp
+Wire Wire Line
+	7950 1800 6050 1800
+Wire Wire Line
+	9450 1300 8050 1300
+Wire Wire Line
+	6050 1600 8050 1600
+Wire Wire Line
+	8050 1300 8050 1600
+Wire Wire Line
+	8150 1400 9450 1400
+Wire Wire Line
+	6050 1700 8150 1700
+Wire Wire Line
+	8150 1400 8150 1700
+Wire Wire Line
+	6050 1500 9450 1500
+Wire Wire Line
+	9450 1750 8300 1750
+Wire Wire Line
+	6050 2000 8300 2000
+Wire Wire Line
+	8300 2000 8300 1750
+$Comp
+L Connector_Generic:Conn_01x02 J101
+U 1 1 5CF0AD96
+P 8150 950
+F 0 "J101" H 8070 625 50  0000 C CNN
+F 1 "AUDIO" H 8070 716 50  0000 C CNN
+F 2 "Pin_Headers:Pin_Header_Straight_1x02_Pitch2.54mm" H 8150 950 50  0001 C CNN
+F 3 "~" H 8150 950 50  0001 C CNN
+	1    8150 950
+	1    0    0    1
+$EndComp
+Wire Wire Line
+	7950 850  7450 850
+Wire Wire Line
+	7450 850  7450 1150
+$Comp
+L power:GND #PWR0126
+U 1 1 5CF15D0B
+P 7800 1250
+F 0 "#PWR0126" H 7800 1000 50  0001 C CNN
+F 1 "GND" H 7805 1077 50  0000 C CNN
+F 2 "" H 7800 1250 50  0001 C CNN
+F 3 "" H 7800 1250 50  0001 C CNN
+	1    7800 1250
+	1    0    0    -1
+$EndComp
+Wire Wire Line
+	7950 950  7800 950
+Wire Wire Line
+	7800 950  7800 1150
+$Comp
+L Mechanical:MountingHole MH101
+U 1 1 5CF43C55
+P 4900 7250
+F 0 "MH101" H 5000 7296 50  0000 L CNN
+F 1 "MountingHole" H 5000 7205 50  0000 L CNN
+F 2 "Mounting_Holes:MountingHole_3.2mm_M3_DIN965" H 4900 7250 50  0001 C CNN
+F 3 "~" H 4900 7250 50  0001 C CNN
+	1    4900 7250
+	1    0    0    -1
+$EndComp
+$Comp
+L Mechanical:MountingHole MH103
+U 1 1 5CF43CF8
+P 4900 7500
+F 0 "MH103" H 5000 7546 50  0000 L CNN
+F 1 "MountingHole" H 5000 7455 50  0000 L CNN
+F 2 "Mounting_Holes:MountingHole_3.2mm_M3_DIN965" H 4900 7500 50  0001 C CNN
+F 3 "~" H 4900 7500 50  0001 C CNN
+	1    4900 7500
+	1    0    0    -1
+$EndComp
+$Comp
+L Mechanical:MountingHole MH102
+U 1 1 5CF43D3E
+P 5650 7250
+F 0 "MH102" H 5750 7296 50  0000 L CNN
+F 1 "MountingHole" H 5750 7205 50  0000 L CNN
+F 2 "Mounting_Holes:MountingHole_3.2mm_M3_DIN965" H 5650 7250 50  0001 C CNN
+F 3 "~" H 5650 7250 50  0001 C CNN
+	1    5650 7250
+	1    0    0    -1
+$EndComp
+$Comp
+L Mechanical:MountingHole MH104
+U 1 1 5CF43D94
+P 5650 7500
+F 0 "MH104" H 5750 7546 50  0000 L CNN
+F 1 "MountingHole" H 5750 7455 50  0000 L CNN
+F 2 "Mounting_Holes:MountingHole_3.2mm_M3_DIN965" H 5650 7500 50  0001 C CNN
+F 3 "~" H 5650 7500 50  0001 C CNN
+	1    5650 7500
+	1    0    0    -1
+$EndComp
+$Comp
+L Device:C_Small C108
+U 1 1 5CF60139
+P 7650 1150
+F 0 "C108" V 7421 1150 50  0000 C CNN
+F 1 "10p" V 7512 1150 50  0000 C CNN
+F 2 "Capacitors_SMD:C_0603_HandSoldering" H 7650 1150 50  0001 C CNN
+F 3 "~" H 7650 1150 50  0001 C CNN
+	1    7650 1150
+	0    1    1    0
+$EndComp
+Wire Wire Line
+	7750 1150 7800 1150
+Connection ~ 7800 1150
+Wire Wire Line
+	7800 1150 7800 1250
+Wire Wire Line
+	7550 1150 7450 1150
+Connection ~ 7450 1150
+Wire Wire Line
+	7450 1150 7450 1400
 $EndSCHEMATC

Commit message: Lots and lots of updates Added DAC amplifier that can be controlled Cleaned up the schematic
Parts:
- removed C107: 10u, Capacitors_SMD:C_0603_HandSoldering, symbol Device:C_Small
- removed C108: 10p, Capacitors_SMD:C_0603_HandSoldering, symbol Device:C_Small
- removed J101: AUDIO, Pin_Headers:Pin_Header_Straight_1x02_Pitch2.54mm, symbol Connector_Generic:Conn_01x02
Connections:
- net labels added: AMP_CS, AMP_DIR, DAC_OUT
- wire segments 153 -> 146
- no-connect marks 6 -> 4
Changed lines of the file:
@@
 Wire Wire Line
 	6050 2700 6150 2700
-Text GLabel 6150 2700 2    50   Output ~ 0
+Text GLabel 6150 3600 2    50   Output ~ 0
 OUT2
 Wire Wire Line
@@
 Text GLabel 6150 2900 2    50   Output ~ 0
 OUT3
-Text GLabel 6150 3600 2    50   Output ~ 0
+Text GLabel 6150 2700 2    50   Output ~ 0
 OUT4
 Text GLabel 6150 2800 2    50   Output ~ 0
@@
 $EndComp
 NoConn ~ 4850 2200
-NoConn ~ 6050 4500
-NoConn ~ 6050 4600
 Wire Wire Line
 	4200 6150 4200 6100
@@
 	10400 1500 10400 1750
 Connection ~ 10400 1750
-$Comp
-L Device:C_Small C107
-U 1 1 5CE9FBD8
-P 7300 1400
-F 0 "C107" V 7071 1400 50  0000 C CNN
-F 1 "10u" V 7162 1400 50  0000 C CNN
-F 2 "Capacitors_SMD:C_0603_HandSoldering" H 7300 1400 50  0001 C CNN
-F 3 "~" H 7300 1400 50  0001 C CNN
-	1    7300 1400
-	0    1    1    0
-$EndComp
-Wire Wire Line
-	7450 1400 7400 1400
-Wire Wire Line
-	6050 1400 7200 1400
+Wire Wire Line
+	6050 1400 6200 1400
 $Comp
 L Misc:IS25LP032D U102
@@
 	8300 2000 8300 1750
 $Comp
-L Connector_Generic:Conn_01x02 J101
-U 1 1 5CF0AD96
-P 8150 950
-F 0 "J101" H 8070 625 50  0000 C CNN
-F 1 "AUDIO" H 8070 716 50  0000 C CNN
-F 2 "Pin_Headers:Pin_Header_Straight_1x02_Pitch2.54mm" H 8150 950 50  0001 C CNN
-F 3 "~" H 8150 950 50  0001 C CNN
-	1    8150 950
-	1    0    0    1
-$EndComp
-Wire Wire Line
-	7950 850  7450 850
-Wire Wire Line
-	7450 850  7450 1150
-$Comp
-L power:GND #PWR0126
-U 1 1 5CF15D0B
-P 7800 1250
-F 0 "#PWR0126" H 7800 1000 50  0001 C CNN
-F 1 "GND" H 7805 1077 50  0000 C CNN
-F 2 "" H 7800 1250 50  0001 C CNN
-F 3 "" H 7800 1250 50  0001 C CNN
-	1    7800 1250
-	1    0    0    -1
-$EndComp
-Wire Wire Line
-	7950 950  7800 950
-Wire Wire Line
-	7800 950  7800 1150
-$Comp
 L Mechanical:MountingHole MH101
 U 1 1 5CF43C55
@@
 	1    0    0    -1
 $EndComp
-$Comp
-L Device:C_Small C108
-U 1 1 5CF60139
-P 7650 1150
-F 0 "C108" V 7421 1150 50  0000 C CNN
-F 1 "10p" V 7512 1150 50  0000 C CNN
-F 2 "Capacitors_SMD:C_0603_HandSoldering" H 7650 1150 50  0001 C CNN
-F 3 "~" H 7650 1150 50  0001 C CNN
-	1    7650 1150
-	0    1    1    0
-$EndComp
-Wire Wire Line
-	7750 1150 7800 1150
-Connection ~ 7800 1150
-Wire Wire Line
-	7800 1150 7800 1250
-Wire Wire Line
-	7550 1150 7450 1150
-Connection ~ 7450 1150
-Wire Wire Line
-	7450 1150 7450 1400
+Text GLabel 6200 1400 2    50   Output ~ 0
+DAC_OUT
+Text GLabel 6150 4500 2    50   Output ~ 0
+AMP_DIR
+Text GLabel 6150 4600 2    50   Output ~ 0
+AMP_CS
+Wire Wire Line
+	6150 4500 6050 4500
+Wire Wire Line
+	6050 4600 6150 4600
 $EndSCHEMATC

Commit message: Added SWD connector for debugging
Parts:
- added TP101: RST, Wire_Pads:SolderWirePad_single_0-8mmDrill, symbol Connector:TestPoint
- added TP102: SWDIO, Wire_Pads:SolderWirePad_single_0-8mmDrill, symbol Connector:TestPoint
- added TP103: SWCLK, Wire_Pads:SolderWirePad_single_0-8mmDrill, symbol Connector:TestPoint
- added TP104: 3V3, Wire_Pads:SolderWirePad_single_0-8mmDrill, symbol Connector:TestPoint
- added TP105: GND, Wire_Pads:SolderWirePad_single_0-8mmDrill, symbol Connector:TestPoint
Connections:
- wire segments 146 -> 152
Changed lines of the file:
@@
 OUT2
 Wire Wire Line
-	6150 2300 6050 2300
+	7350 2300 6850 2300
 Text GLabel 6150 3300 2    50   Output ~ 0
 HC_OUT1
 Text GLabel 6150 3400 2    50   Output ~ 0
 HC_OUT2
-Text GLabel 6150 2300 2    50   Output ~ 0
+Text GLabel 7350 2300 2    50   Output ~ 0
 OUT1
 Wire Wire Line
@@
 	7950 1200 7950 1800
 Wire Wire Line
-	6050 2400 8300 2400
+	6050 2400 7850 2400
 Wire Wire Line
 	8300 2400 8300 3850
@@
 Wire Wire Line
 	6050 4600 6150 4600
+$Comp
+L Connector:TestPoint TP102
+U 1 1 5CECADFA
+P 6850 2300
+F 0 "TP102" H 6908 2420 50  0000 L CNN
+F 1 "SWDIO" H 6908 2329 50  0000 L CNN
+F 2 "Wire_Pads:SolderWirePad_single_0-8mmDrill" H 7050 2300 50  0001 C CNN
+F 3 "~" H 7050 2300 50  0001 C CNN
+	1    6850 2300
+	1    0    0    -1
+$EndComp
+$Comp
+L Connector:TestPoint TP103
+U 1 1 5CECB040
+P 7850 2400
+F 0 "TP103" H 7908 2520 50  0000 L CNN
+F 1 "SWCLK" H 7908 2429 50  0000 L CNN
+F 2 "Wire_Pads:SolderWirePad_single_0-8mmDrill" H 8050 2400 50  0001 C CNN
+F 3 "~" H 8050 2400 50  0001 C CNN
+	1    7850 2400
+	1    0    0    -1
+$EndComp
+Connection ~ 7850 2400
+Wire Wire Line
+	7850 2400 8300 2400
+Connection ~ 6850 2300
+Wire Wire Line
+	6850 2300 6050 2300
+$Comp
+L Connector:TestPoint TP101
+U 1 1 5CED0971
+P 4800 850
+F 0 "TP101" H 4858 970 50  0000 L CNN
+F 1 "RST" H 4858 879 50  0000 L CNN
+F 2 "Wire_Pads:SolderWirePad_single_0-8mmDrill" H 5000 850 50  0001 C CNN
+F 3 "~" H 5000 850 50  0001 C CNN
+	1    4800 850
+	1    0    0    -1
+$EndComp
+Connection ~ 4800 850
+$Comp
+L Connector:TestPoint TP104
+U 1 1 5CED1B66
+P 4000 3300
+F 0 "TP104" H 4058 3420 50  0000 L CNN
+F 1 "3V3" H 4058 3329 50  0000 L CNN
+F 2 "Wire_Pads:SolderWirePad_single_0-8mmDrill" H 4200 3300 50  0001 C CNN
+F 3 "~" H 4200 3300 50  0001 C CNN
+	1    4000 3300
+	1    0    0    -1
+$EndComp
+$Comp
+L power:+3V3 #PWR0126
+U 1 1 5CED1EA6
+P 3800 3300
+F 0 "#PWR0126" H 3800 3150 50  0001 C CNN
+F 1 "+3V3" H 3815 3473 50  0000 C CNN
+F 2 "" H 3800 3300 50  0001 C CNN
+F 3 "" H 3800 3300 50  0001 C CNN
+	1    3800 3300
+	1    0    0    -1
+$EndComp
+Wire Wire Line
+	4000 3300 4000 3350
+Wire Wire Line
+	4000 3350 3800 3350
+Wire Wire Line
+	3800 3350 3800 3300
+$Comp
+L Connector:TestPoint TP105
+U 1 1 5CED7BFF
+P 4000 3600
+F 0 "TP105" H 4058 3720 50  0000 L CNN
+F 1 "GND" H 4058 3629 50  0000 L CNN
+F 2 "Wire_Pads:SolderWirePad_single_0-8mmDrill" H 4200 3600 50  0001 C CNN
+F 3 "~" H 4200 3600 50  0001 C CNN
+	1    4000 3600
+	1    0    0    -1
+$EndComp
+$Comp
+L power:GND #PWR0127
+U 1 1 5CED7C70
+P 4000 3650
+F 0 "#PWR0127" H 4000 3400 50  0001 C CNN
+F 1 "GND" H 4005 3477 50  0000 C CNN
+F 2 "" H 4000 3650 50  0001 C CNN
+F 3 "" H 4000 3650 50  0001 C CNN
+	1    4000 3650
+	1    0    0    -1
+$EndComp
+Wire Wire Line
+	4000 3600 4000 3650
 $EndSCHEMATC

Commit message: Changed the digital potentiometer to AD5160 10k version and enabled SPI3
Parts:
- removed X101: TXC-7C, PCBDecals:IQXO-791, symbol Oscillator:TXC-7C
- added X101: SG-310_SCF_8.000000MHZ, PCBDecals:SG- 310, symbol Misc:SG-310_SCF_8.000000MHZ
- J105: footprint Connect:USB_Micro-B -> PCBDecals:USB_Micro-B
- U102: footprint digikey-footprints:SOIC-8_W3.9mm -> digikey-footprints:SOIC-8_W5.6mm
Connections:
- net labels added: AMP_CLK, AMP_DIN
- wire segments 152 -> 151
- no-connect marks 4 -> 2
Changed lines of the file:
@@
 U 1 1 5CE1FC54
 P 4600 1400
-F 0 "R102" H 4500 1400 50  0000 C CNN
+F 0 "R102" H 4750 1500 50  0000 C CNN
 F 1 "470R" V 4600 1400 50  0000 C CNN
 F 2 "Resistors_SMD:R_0603_HandSoldering" V 4530 1400 50  0001 C CNN
@@
 F 0 "J105" H 3855 6817 50  0000 C CNN
 F 1 "USB_B_Micro" H 3855 6726 50  0000 C CNN
-F 2 "Connect:USB_Micro-B" H 3950 6300 50  0001 C CNN
+F 2 "PCBDecals:USB_Micro-B" H 3950 6300 50  0001 C CNN
 F 3 "~" H 3950 6300 50  0001 C CNN
 	1    3800 6350
@@
 Wire Wire Line
 	3600 2000 3550 2000
-Wire Wire Line
-	3550 2000 3550 1650
-Wire Wire Line
-	3550 1650 3900 1650
 Connection ~ 3900 1650
 Wire Wire Line
@@
 $EndComp
 Wire Wire Line
-	3550 1650 3450 1650
-Wire Wire Line
 	3450 1650 3450 2150
-Connection ~ 3550 1650
 Wire Wire Line
 	3900 2400 3450 2400
@@
 L power:GND #PWR0104
 U 1 1 5CE4C56B
-P 10400 1800
-F 0 "#PWR0104" H 10400 1550 50  0001 C CNN
-F 1 "GND" H 10405 1627 50  0000 C CNN
-F 2 "" H 10400 1800 50  0001 C CNN
-F 3 "" H 10400 1800 50  0001 C CNN
-	1    10400 1800
+P 10400 1850
+F 0 "#PWR0104" H 10400 1600 50  0001 C CNN
+F 1 "GND" H 10405 1677 50  0000 C CNN
+F 2 "" H 10400 1850 50  0001 C CNN
+F 3 "" H 10400 1850 50  0001 C CNN
+	1    10400 1850
 	1    0    0    -1
 $EndComp
@@
 Text GLabel 6150 2500 2    50   Output ~ 0
 SERVO_OUT1
-Text GLabel 6150 3000 2    50   Output ~ 0
+Text GLabel 6150 3100 2    50   Output ~ 0
 SERVO_OUT2
 Text GLabel 6150 4200 2    50   Output ~ 0
@@
 Text GLabel 6150 2800 2    50   Output ~ 0
 OUT5
-Text GLabel 6150 3100 2    50   Output ~ 0
+Text GLabel 6150 3500 2    50   Output ~ 0
 OUT6
 Wire Wire Line
@@
 Wire Wire Line
 	4100 6150 4200 6150
-$Comp
-L Oscillator:TXC-7C X101
-U 1 1 5CE6962F
-P 3900 2000
-F 0 "X101" H 4241 2046 50  0000 L CNN
-F 1 "TXC-7C" H 4241 1955 50  0000 L CNN
-F 2 "PCBDecals:IQXO-791" H 4600 1650 50  0001 C CNN
-F 3 "http://www.txccorp.com/download/products/osc/7C_o.pdf" H 3800 2000 50  0001 C CNN
-	1    3900 2000
-	1    0    0    -1
-$EndComp
 NoConn ~ 4850 2200
 Wire Wire Line
@@
 COOLING_TEMP
 Wire Wire Line
-	7950 1200 7950 1800
+	8250 1200 8250 1800
 Wire Wire Line
 	6050 2400 7850 2400
@@
 Connection ~ 9000 3850
 Wire Wire Line
-	7950 1200 9450 1200
-Wire Wire Line
-	10350 1750 10400 1750
-Wire Wire Line
-	10400 1750 10400 1800
+	8250 1200 9500 1200
 $Comp
 L power:+3V3 #PWR0101
 U 1 1 5CEF7FBB
-P 9400 750
-F 0 "#PWR0101" H 9400 600 50  0001 C CNN
-F 1 "+3V3" H 9415 923 50  0000 C CNN
-F 2 "" H 9400 750 50  0001 C CNN
-F 3 "" H 9400 750 50  0001 C CNN
-	1    9400 750
-	1    0    0    -1
-$EndComp
-Wire Wire Line
-	9450 1050 9400 1050
-Wire Wire Line
-	9400 1050 9400 750
+P 9500 700
+F 0 "#PWR0101" H 9500 550 50  0001 C CNN
+F 1 "+3V3" H 9515 873 50  0000 C CNN
+F 2 "" H 9500 700 50  0001 C CNN
+F 3 "" H 9500 700 50  0001 C CNN
+	1    9500 700
+	1    0    0    -1
+$EndComp
 Text Label 8550 1750 0    50   ~ 0
 WP
-NoConn ~ 9450 1650
-NoConn ~ 6050 3500
-NoConn ~ 6050 3200
+NoConn ~ 9500 1650
 $Comp
 L Device:LED D101
@@
 	10400 1300 10400 750
 Wire Wire Line
-	10400 750  9400 750
-Connection ~ 9400 750
-Wire Wire Line
-	10400 1500 10400 1750
-Connection ~ 10400 1750
-Wire Wire Line
 	6050 1400 6200 1400
-$Comp
-L Misc:IS25LP032D U102
-U 1 1 5CEB0F5A
-P 9900 1400
-F 0 "U102" H 9900 1975 50  0000 C CNN
-F 1 "IS25LP032D" H 9900 1884 50  0000 C CNN
-F 2 "digikey-footprints:SOIC-8_W3.9mm" H 9800 1250 50  0001 C CNN
-F 3 "" H 9800 1250 50  0001 C CNN
-	1    9900 1400
-	1    0    0    -1
-$EndComp
-Wire Wire Line
-	7950 1800 6050 1800
-Wire Wire Line
-	9450 1300 8050 1300
+Wire Wire Line
+	8250 1800 6050 1800
 Wire Wire Line
 	6050 1600 8050 1600
@@
 	8050 1300 8050 1600
 Wire Wire Line
-	8150 1400 9450 1400
+	8150 1400 9500 1400
 Wire Wire Line
 	6050 1700 8150 1700
@@
 	8150 1400 8150 1700
 Wire Wire Line
-	6050 1500 9450 1500
-Wire Wire Line
-	9450 1750 8300 1750
-Wire Wire Line
-	6050 2000 8300 2000
-Wire Wire Line
-	8300 2000 8300 1750
+	6050 1500 9500 1500
+Wire Wire Line
+	9500 1750 8350 1750
+Wire Wire Line
+	6050 2000 8350 2000
+Wire Wire Line
+	8350 2000 8350 1750
 $Comp
 L Mechanical:MountingHole MH101
@@
 Wire Wire Line
 	4000 3600 4000 3650
+$Comp
+L Misc:SG-310_SCF_8.000000MHZ X101
+U 1 1 5CECEA0C
+P 3900 2000
+F 0 "X101" H 3950 2250 50  0000 L CNN
+F 1 "SG-310_SCF_8.000000MHZ" H 4450 1750 50  0001 C CNN
+F 2 "PCBDecals:SG- 310" H 3900 2000 50  0001 C CNN
+F 3 "https://support.epson.biz/td/api/doc_check.php?dl=brief_SG-310SEF&lang=en" H 3900 2000 50  0001 C CNN
+	1    3900 2000
+	1    0    0    -1
+$EndComp
+Wire Wire Line
+	3450 1650 3900 1650
+Wire Wire Line
+	8050 1300 9500 1300
+Wire Wire Line
+	10400 1500 10400 1750
+$Comp
+L Misc:IS25LP032D U102
+U 1 1 5CF328C7
+P 9950 1400
+F 0 "U102" H 9950 1975 50  0000 C CNN
+F 1 "IS25LP032D" H 9950 1884 50  0000 C CNN
+F 2 "digikey-footprints:SOIC-8_W5.6mm" H 9850 1250 50  0001 C CNN
+F 3 "http://www.issi.com/WW/pdf/25LP-WP032D.pdf" H 9850 1250 50  0001 C CNN
+	1    9950 1400
+	1    0    0    -1
+$EndComp
+Connection ~ 10400 1750
+Wire Wire Line
+	10400 1750 10400 1850
+Wire Wire Line
+	9500 750  10400 750
+Wire Wire Line
+	9500 700  9500 750
+Connection ~ 9500 750
+Wire Wire Line
+	9500 750  9500 1050
+Wire Wire Line
+	6150 3500 6050 3500
+Wire Wire Line
+	6050 3200 6150 3200
+Text GLabel 6150 3000 2    50   Output ~ 0
+AMP_CLK
+Text GLabel 6150 3200 2    50   Output ~ 0
+AMP_DIN
 $EndSCHEMATC

Commit message: Refactored schematic net names
Connections:
- net labels added: SERVO_1, SERVO_2, SERVO_3, SERVO_4
- net labels removed: SERVO_OUT1, SERVO_OUT2, SERVO_OUT3, SERVO_OUT4
Changed lines of the file:
@@
 SPI_CS
 Text GLabel 6150 2500 2    50   Output ~ 0
-SERVO_OUT1
+SERVO_1
 Text GLabel 6150 3100 2    50   Output ~ 0
-SERVO_OUT2
+SERVO_2
 Text GLabel 6150 4200 2    50   Output ~ 0
-SERVO_OUT3
+SERVO_3
 Text GLabel 6150 4100 2    50   Output ~ 0
-SERVO_OUT4
+SERVO_4
 Wire Wire Line
 	6150 2500 6050 2500

Commit message: Renamed schematic pdf Added gerbers Added layout pdf Fixed silkscreen on layout
Changed lines of the file:
@@
 L power:+3V3 #PWR0125
 U 1 1 5CF145CC
-P 7450 4300
-F 0 "#PWR0125" H 7450 4150 50  0001 C CNN
-F 1 "+3V3" H 7465 4473 50  0000 C CNN
-F 2 "" H 7450 4300 50  0001 C CNN
-F 3 "" H 7450 4300 50  0001 C CNN
-	1    7450 4300
+P 7650 4300
+F 0 "#PWR0125" H 7650 4150 50  0001 C CNN
+F 1 "+3V3" H 7665 4473 50  0000 C CNN
+F 2 "" H 7650 4300 50  0001 C CNN
+F 3 "" H 7650 4300 50  0001 C CNN
+	1    7650 4300
 	1    0    0    -1
 $EndComp
 Wire Wire Line
-	7450 4300 7450 4400
+	7650 4300 7650 4400
 Wire Wire Line
-	7450 4400 7250 4400
+	7650 4400 7250 4400
 $Comp
 L Misc:STM32F303CBx U101

Commit message: Added cooling temperature sensor
Parts:
- added J101: BOOT0, Pin_Headers:Pin_Header_Straight_1x02_Pitch1.27mm, symbol Connector_Generic:Conn_01x02
- added R104: 10k, Resistors_SMD:R_0603_HandSoldering, symbol Device:R_Small
Connections:
- net labels removed: AMP_DIR
- wire segments 151 -> 156
- no-connect marks 2 -> 5
Changed lines of the file:
@@
 	8900 2750 8900 2800
 Wire Wire Line
-	4100 6150 4200 6150
+	4100 6150 4350 6150
 NoConn ~ 4850 2200
 Wire Wire Line
-	4200 6150 4200 6100
+	4350 6150 4350 6100
 $Comp
 L power:VBUS #PWR0112
 U 1 1 5CEEB052
-P 4200 6100
-F 0 "#PWR0112" H 4200 5950 50  0001 C CNN
-F 1 "VBUS" H 4215 6273 50  0000 C CNN
-F 2 "" H 4200 6100 50  0001 C CNN
-F 3 "" H 4200 6100 50  0001 C CNN
-	1    4200 6100
+P 4350 6100
+F 0 "#PWR0112" H 4350 5950 50  0001 C CNN
+F 1 "VBUS" H 4365 6273 50  0000 C CNN
+F 2 "" H 4350 6100 50  0001 C CNN
+F 3 "" H 4350 6100 50  0001 C CNN
+	1    4350 6100
 	1    0    0    -1
 $EndComp
@@
 Text GLabel 6200 1400 2    50   Output ~ 0
 DAC_OUT
-Text GLabel 6150 4500 2    50   Output ~ 0
-AMP_DIR
 Text GLabel 6150 4600 2    50   Output ~ 0
 AMP_CS
-Wire Wire Line
-	6150 4500 6050 4500
 Wire Wire Line
 	6050 4600 6150 4600
@@
 Text GLabel 6150 3200 2    50   Output ~ 0
 AMP_DIN
+NoConn ~ 6050 4500
+NoConn ~ 4100 6550
+NoConn ~ 3550 2000
+$Comp
+L Connector_Generic:Conn_01x02 J101
+U 1 1 5CF7480D
+P 6650 6100
+F 0 "J101" H 6570 5775 50  0000 C CNN
+F 1 "BOOT0" H 6570 5866 50  0000 C CNN
+F 2 "Pin_Headers:Pin_Header_Straight_1x02_Pitch1.27mm" H 6650 6100 50  0001 C CNN
+F 3 "~" H 6650 6100 50  0001 C CNN
+	1    6650 6100
+	1    0    0    -1
+$EndComp
+Text GLabel 6250 6100 0    50   Input ~ 0
+COOLING_TEMP
+$Comp
+L Device:R_Small R104
+U 1 1 5CF74AE7
+P 6400 5850
+F 0 "R104" H 6459 5896 50  0000 L CNN
+F 1 "10k" H 6459 5805 50  0000 L CNN
+F 2 "Resistors_SMD:R_0603_HandSoldering" H 6400 5850 50  0001 C CNN
+F 3 "~" H 6400 5850 50  0001 C CNN
+	1    6400 5850
+	1    0    0    -1
+$EndComp
+Wire Wire Line
+	6250 6100 6400 6100
+Wire Wire Line
+	6400 5950 6400 6100
+Connection ~ 6400 6100
+Wire Wire Line
+	6400 6100 6450 6100
+Wire Wire Line
+	6400 5700 6400 5750
+Wire Wire Line
+	6450 6200 6400 6200
+Wire Wire Line
+	6400 6200 6400 6450
+$Comp
+L power:GND #PWR0130
+U 1 1 5CF8CD64
+P 6400 6450
+F 0 "#PWR0130" H 6400 6200 50  0001 C CNN
+F 1 "GND" H 6405 6277 50  0000 C CNN
+F 2 "" H 6400 6450 50  0001 C CNN
+F 3 "" H 6400 6450 50  0001 C CNN
+	1    6400 6450
+	1    0    0    -1
+$EndComp
+$Comp
+L power:+3V3 #PWR0129
+U 1 1 5CF8CEC5
+P 6400 5700
+F 0 "#PWR0129" H 6400 5550 50  0001 C CNN
+F 1 "+3V3" H 6415 5873 50  0000 C CNN
+F 2 "" H 6400 5700 50  0001 C CNN
+F 3 "" H 6400 5700 50  0001 C CNN
+	1    6400 5700
+	1    0    0    -1
+$EndComp
 $EndSCHEMATC
