File: hw/Telemetry.sch (KiCad schematic (older format))
At the start: 31 parts, among them J101 BOOT0, J102 BOOT0, J103 SPORT, J104 SBUS, J105 USB_B_Micro, J106 UART_EXP, SW101 SW_Push, U101 STM32F303CBx, U102 IS25LP032D, X101 SG-310_SCF_8.000000MHZ

Commit message: Added Opto-isolated inputs to the design Added uartdriver to the project Refined pin definitions
Parts:
- J103, J104: footprint Pin_Headers:Pin_Header_Angled_2x03 -> Pin_Headers:Pin_Header_Straight_2x03
Connections:
- net labels added: HC_PWM1, HC_PWM2, IN1, IN2, PWM1, PWM2
- net labels removed: HC_OUT1, HC_OUT2, OUT3, OUT4, OUT5, OUT6
Changed lines of the file:
@@
 L Connector_Generic:Conn_01x06 J103
 U 1 1 5CE7FF53
-P 9250 3300
-F 0 "J103" H 9329 3292 50  0000 L CNN
-F 1 "SPORT" H 9329 3201 50  0000 L CNN
-F 2 "Pin_Headers:Pin_Header_Angled_2x03" H 9250 3300 50  0001 C CNN
-F 3 "~" H 9250 3300 50  0001 C CNN
-	1    9250 3300
+P 9250 2600
+F 0 "J103" H 9329 2592 50  0000 L CNN
+F 1 "SPORT" H 9329 2501 50  0000 L CNN
+F 2 "Pin_Headers:Pin_Header_Straight_2x03" H 9250 2600 50  0001 C CNN
+F 3 "~" H 9250 2600 50  0001 C CNN
+	1    9250 2600
 	1    0    0    -1
 $EndComp
@@
 L power:VCC #PWR0105
 U 1 1 5CE8046C
-P 8900 2750
-F 0 "#PWR0105" H 8900 2600 50  0001 C CNN
-F 1 "VCC" H 8917 2923 50  0000 C CNN
-F 2 "" H 8900 2750 50  0001 C CNN
-F 3 "" H 8900 2750 50  0001 C CNN
-	1    8900 2750
-	1    0    0    -1
-$EndComp
-Wire Wire Line
-	9050 3300 8900 3300
-Wire Wire Line
-	9050 3400 8900 3400
-Wire Wire Line
-	8900 3400 8900 3300
-Wire Wire Line
-	9050 3500 8800 3500
-Wire Wire Line
-	8800 3500 8800 3600
-Wire Wire Line
-	9050 3600 8800 3600
-Connection ~ 8800 3600
-Wire Wire Line
-	9050 3200 9000 3200
-Wire Wire Line
-	9000 3200 9000 3100
-Wire Wire Line
-	9000 3100 9050 3100
+P 8900 2050
+F 0 "#PWR0105" H 8900 1900 50  0001 C CNN
+F 1 "VCC" H 8917 2223 50  0000 C CNN
+F 2 "" H 8900 2050 50  0001 C CNN
+F 3 "" H 8900 2050 50  0001 C CNN
+	1    8900 2050
+	1    0    0    -1
+$EndComp
+Wire Wire Line
+	9050 2600 8900 2600
+Wire Wire Line
+	9050 2700 8900 2700
+Wire Wire Line
+	8900 2700 8900 2600
+Wire Wire Line
+	9050 2800 8800 2800
+Wire Wire Line
+	8800 2800 8800 2900
+Wire Wire Line
+	9050 2900 8800 2900
+Connection ~ 8800 2900
+Wire Wire Line
+	9050 2500 9000 2500
+Wire Wire Line
+	9000 2500 9000 2400
+Wire Wire Line
+	9000 2400 9050 2400
 $Comp
 L Connector_Generic:Conn_01x06 J104
 U 1 1 5CEA038E
-P 9250 4050
-F 0 "J104" H 9329 4042 50  0000 L CNN
-F 1 "SBUS" H 9329 3951 50  0000 L CNN
-F 2 "Pin_Headers:Pin_Header_Angled_2x03" H 9250 4050 50  0001 C CNN
-F 3 "~" H 9250 4050 50  0001 C CNN
-	1    9250 4050
+P 9250 3350
+F 0 "J104" H 9329 3342 50  0000 L CNN
+F 1 "SBUS" H 9329 3251 50  0000 L CNN
+F 2 "Pin_Headers:Pin_Header_Straight_2x03" H 9250 3350 50  0001 C CNN
+F 3 "~" H 9250 3350 50  0001 C CNN
+	1    9250 3350
 	1    0    0    -1
 $EndComp
@@
 L power:GND #PWR0109
 U 1 1 5CEA03A3
-P 8800 4450
-F 0 "#PWR0109" H 8800 4200 50  0001 C CNN
-F 1 "GND" H 8805 4277 50  0000 C CNN
-F 2 "" H 8800 4450 50  0001 C CNN
-F 3 "" H 8800 4450 50  0001 C CNN
-	1    8800 4450
-	1    0    0    -1
-$EndComp
-Wire Wire Line
-	9050 4050 8900 4050
-Wire Wire Line
-	9050 4150 8900 4150
-Wire Wire Line
-	8900 4150 8900 4050
-Connection ~ 8900 4050
-Wire Wire Line
-	9050 4250 8800 4250
-Wire Wire Line
-	9050 4350 8800 4350
-Connection ~ 8800 4350
-Wire Wire Line
-	8800 4350 8800 4450
-Wire Wire Line
-	9050 3950 9000 3950
-Wire Wire Line
-	9000 3950 9000 3850
-Wire Wire Line
-	9000 3850 9050 3850
+P 8800 3750
+F 0 "#PWR0109" H 8800 3500 50  0001 C CNN
+F 1 "GND" H 8805 3577 50  0000 C CNN
+F 2 "" H 8800 3750 50  0001 C CNN
+F 3 "" H 8800 3750 50  0001 C CNN
+	1    8800 3750
+	1    0    0    -1
+$EndComp
+Wire Wire Line
+	9050 3350 8900 3350
+Wire Wire Line
+	9050 3450 8900 3450
+Wire Wire Line
+	8900 3450 8900 3350
+Connection ~ 8900 3350
+Wire Wire Line
+	9050 3550 8800 3550
+Wire Wire Line
+	9050 3650 8800 3650
+Connection ~ 8800 3650
+Wire Wire Line
+	8800 3650 8800 3750
+Wire Wire Line
+	9050 3250 9000 3250
+Wire Wire Line
+	9000 3250 9000 3150
+Wire Wire Line
+	9000 3150 9050 3150
 Wire Wire Line
 	6050 2100 6400 2100
@@
 Wire Wire Line
 	3900 2400 3900 2450
-Text Label 8550 3850 0    50   ~ 0
+Text Label 8550 3150 0    50   ~ 0
 Sbus
-Connection ~ 9000 3100
-Text Label 8500 3100 0    50   ~ 0
+Connection ~ 9000 2400
+Text Label 8500 2400 0    50   ~ 0
 S.port
 Wire Wire Line
-	8450 3100 8450 1900
+	8450 2400 8450 1900
 Wire Wire Line
 	8450 1900 6050 1900
 Wire Wire Line
-	8450 3100 9000 3100
+	8450 2400 9000 2400
 $Comp
 L power:GND #PWR0104
@@
 $EndComp
 Wire Wire Line
-	8900 3400 8900 4050
-Connection ~ 8900 3400
-Wire Wire Line
-	8800 3600 8800 4250
-Connection ~ 8800 4250
-Wire Wire Line
-	8800 4250 8800 4350
+	8900 2700 8900 3350
+Connection ~ 8900 2700
+Wire Wire Line
+	8800 2900 8800 3550
+Connection ~ 8800 3550
+Wire Wire Line
+	8800 3550 8800 3650
 $Comp
 L Switch:SW_Push SW101
@@
 	6050 2700 6150 2700
 Text GLabel 6150 3600 2    50   Output ~ 0
-OUT2
+PWM2
 Wire Wire Line
 	7350 2300 6850 2300
 Text GLabel 6150 3300 2    50   Output ~ 0
-HC_OUT1
+HC_PWM1
 Text GLabel 6150 3400 2    50   Output ~ 0
-HC_OUT2
+HC_PWM2
 Text GLabel 7350 2300 2    50   Output ~ 0
-OUT1
+PWM1
 Wire Wire Line
 	6150 3300 6050 3300
@@
 	6150 3600 6050 3600
 Text GLabel 6150 2900 2    50   Output ~ 0
-OUT3
-Text GLabel 6150 2700 2    50   Output ~ 0
-OUT4
+OUT1
+Text GLabel 6150 2700 2    50   Input ~ 0
+IN1
 Text GLabel 6150 2800 2    50   Output ~ 0
-OUT5
-Text GLabel 6150 3500 2    50   Output ~ 0
-OUT6
+OUT2
+Text GLabel 6150 3500 2    50   Input ~ 0
+IN2
 Wire Wire Line
 	6050 2800 6150 2800
@@
 L Device:Jumper_NC_Small JP101
 U 1 1 5CE9AC78
-P 8900 2900
-F 0 "JP101" V 8946 2853 50  0000 R CNN
-F 1 "Jumper_NC_Small" V 8855 2853 50  0000 R CNN
-F 2 "Pin_Headers:Pin_Header_Straight_1x02" H 8900 2900 50  0001 C CNN
-F 3 "~" H 8900 2900 50  0001 C CNN
-	1    8900 2900
+P 8900 2200
+F 0 "JP101" V 8946 2153 50  0000 R CNN
+F 1 "Jumper_NC_Small" V 8855 2153 50  0000 R CNN
+F 2 "Pin_Headers:Pin_Header_Straight_1x02" H 8900 2200 50  0001 C CNN
+F 3 "~" H 8900 2200 50  0001 C CNN
+	1    8900 2200
 	0    -1   -1   0
 $EndComp
 Wire Wire Line
-	8900 3000 8900 3300
-Connection ~ 8900 3300
-Wire Wire Line
-	8900 2750 8900 2800
+	8900 2300 8900 2600
+Connection ~ 8900 2600
+Wire Wire Line
+	8900 2050 8900 2100
 Wire Wire Line
 	4100 6150 4350 6150
@@
 	6050 2400 7850 2400
 Wire Wire Line
-	8300 2400 8300 3850
-Wire Wire Line
-	8300 3850 9000 3850
-Connection ~ 9000 3850
+	8300 2400 8300 3150
+Wire Wire Line
+	8300 3150 9000 3150
+Connection ~ 9000 3150
 Wire Wire Line
 	8250 1200 9500 1200
@@
 L Connector:TestPoint TP104
 U 1 1 5CED1B66
-P 4000 3300
-F 0 "TP104" H 4058 3420 50  0000 L CNN
-F 1 "3V3" H 4058 3329 50  0000 L CNN
-F 2 "Wire_Pads:SolderWirePad_single_0-8mmDrill" H 4200 3300 50  0001 C CNN
-F 3 "~" H 4200 3300 50  0001 C CNN
-	1    4000 3300
+P 2450 7250
+F 0 "TP104" H 2508 7370 50  0000 L CNN
+F 1 "3V3" H 2508 7279 50  0000 L CNN
+F 2 "Wire_Pads:SolderWirePad_single_0-8mmDrill" H 2650 7250 50  0001 C CNN
+F 3 "~" H 2650 7250 50  0001 C CNN
+	1    2450 7250
 	1    0    0    -1
 $EndComp
@@
 L power:+3V3 #PWR0126
 U 1 1 5CED1EA6
-P 3800 3300
-F 0 "#PWR0126" H 3800 3150 50  0001 C CNN
-F 1 "+3V3" H 3815 3473 50  0000 C CNN
-F 2 "" H 3800 3300 50  0001 C CNN
-F 3 "" H 3800 3300 50  0001 C CNN
-	1    3800 3300
-	1    0    0    -1
-$EndComp
-Wire Wire Line
-	4000 3300 4000 3350
-Wire Wire Line
-	4000 3350 3800 3350
-Wire Wire Line
-	3800 3350 3800 3300
+P 2250 7250
+F 0 "#PWR0126" H 2250 7100 50  0001 C CNN
+F 1 "+3V3" H 2265 7423 50  0000 C CNN
+F 2 "" H 2250 7250 50  0001 C CNN
+F 3 "" H 2250 7250 50  0001 C CNN
+	1    2250 7250
+	1    0    0    -1
+$EndComp
+Wire Wire Line
+	2450 7250 2450 7300
+Wire Wire Line
+	2450 7300 2250 7300
+Wire Wire Line
+	2250 7300 2250 7250
 $Comp
 L Connector:TestPoint TP105
 U 1 1 5CED7BFF
-P 4000 3600
-F 0 "TP105" H 4058 3720 50  0000 L CNN
-F 1 "GND" H 4058 3629 50  0000 L CNN
-F 2 "Wire_Pads:SolderWirePad_single_0-8mmDrill" H 4200 3600 50  0001 C CNN
-F 3 "~" H 4200 3600 50  0001 C CNN
-	1    4000 3600
+P 2850 7250
+F 0 "TP105" H 2908 7370 50  0000 L CNN
+F 1 "GND" H 2908 7279 50  0000 L CNN
+F 2 "Wire_Pads:SolderWirePad_single_0-8mmDrill" H 3050 7250 50  0001 C CNN
+F 3 "~" H 3050 7250 50  0001 C CNN
+	1    2850 7250
 	1    0    0    -1
 $EndComp
@@
 L power:GND #PWR0127
 U 1 1 5CED7C70
-P 4000 3650
-F 0 "#PWR0127" H 4000 3400 50  0001 C CNN
-F 1 "GND" H 4005 3477 50  0000 C CNN
-F 2 "" H 4000 3650 50  0001 C CNN
-F 3 "" H 4000 3650 50  0001 C CNN
-	1    4000 3650
-	1    0    0    -1
-$EndComp
-Wire Wire Line
-	4000 3600 4000 3650
+P 2850 7300
+F 0 "#PWR0127" H 2850 7050 50  0001 C CNN
+F 1 "GND" H 2855 7127 50  0000 C CNN
+F 2 "" H 2850 7300 50  0001 C CNN
+F 3 "" H 2850 7300 50  0001 C CNN
+	1    2850 7300
+	1    0    0    -1
+$EndComp
+Wire Wire Line
+	2850 7250 2850 7300
 $Comp
 L Misc:SG-310_SCF_8.000000MHZ X101
