File: hw/Telemetry.sch (KiCad schematic (older format))
At the start: 39 parts, among them J102 BOOT0, J103 SPORT, J104 SBUS, J105 USB_B_Micro, J106 UART_EXP, SW101 SW_Push, U101 STM32F303CBx, U102 IS25LP032D, X101 SG-310_SCF_8.000000MHZ

Commit message: Signal remapping for Flash Memory and component optimizations
Parts:
- U101: symbol Telemetry-rescue:STM32F303CBx-Misc -> Telemetry-rescue:STM32F303CBx-Misc-Telemetry-rescue
- U102: symbol Telemetry-rescue:IS25LP032D-Misc -> Telemetry-rescue:IS25LP032D-Misc-Telemetry-rescue
- X101: symbol Telemetry-rescue:SG-310_SCF_8.000000MHZ-Misc -> Telemetry-rescue:SG-310_SCF_8.000000MHZ-Misc-Telemetry-rescue
Connections:
- net at R103.2: now also U101.4 (PC15); no longer U101.2 (PC13)
- net FLASH_HOLD: now reaches U102.7 (~HOLD/RST)
- net FLASH_HOLD: now also U101.29 (PA8)
- net SPI_CS renamed FLASH_CS
- net FLASH_CS: now also U101.2 (PC13); no longer U101.29 (PA8)
- net SPI_MISO renamed FLASH_MISO
- net SPI_MOSI renamed FLASH_MOSI
- net SPI_SCK renamed FLASH_SCK
- net WP renamed FLASH_WP
- no-connect marks 6 -> 4
Other:
- moved on the sheet: D101, R103
Changed lines of the file:
@@
 F1 "output.sch" 50
 $EndSheet
-Text Label 8550 1500 0    50   ~ 0
-SPI_SCK
-Text Label 8550 1300 0    50   ~ 0
-SPI_MISO
-Text Label 8550 1400 0    50   ~ 0
-SPI_MOSI
-Text Label 8550 1200 0    50   ~ 0
-SPI_CS
 Wire Wire Line
 	6150 2500 6050 2500
@@
 Wire Wire Line
 	6050 4000 6150 4000
-Wire Wire Line
-	8250 1200 8250 1800
 Connection ~ 9000 3700
-Wire Wire Line
-	8250 1200 9500 1200
 $Comp
 L power:+3V3 #PWR0101
@@
 	1    0    0    -1
 $EndComp
-NoConn ~ 9500 1650
 $Comp
 L Device:LED D101
 U 1 1 5CF14422
-P 7100 4400
-F 0 "D101" H 7091 4616 50  0000 C CNN
-F 1 "LED_Green" H 7091 4525 50  0000 C CNN
-F 2 "LEDs:LED_0603_HandSoldering" H 7100 4400 50  0001 C CNN
-F 3 "~" H 7100 4400 50  0001 C CNN
-	1    7100 4400
+P 6800 4600
+F 0 "D101" H 6791 4816 50  0000 C CNN
+F 1 "LED_Green" H 6791 4725 50  0000 C CNN
+F 2 "LEDs:LED_0603_HandSoldering" H 6800 4600 50  0001 C CNN
+F 3 "~" H 6800 4600 50  0001 C CNN
+	1    6800 4600
 	1    0    0    -1
 $EndComp
@@
 L power:+3V3 #PWR0125
 U 1 1 5CF145CC
-P 7650 4300
-F 0 "#PWR0125" H 7650 4150 50  0001 C CNN
-F 1 "+3V3" H 7665 4473 50  0000 C CNN
-F 2 "" H 7650 4300 50  0001 C CNN
-F 3 "" H 7650 4300 50  0001 C CNN
-	1    7650 4300
-	1    0    0    -1
-$EndComp
-Wire Wire Line
-	7650 4300 7650 4400
-Wire Wire Line
-	7650 4400 7250 4400
-$Comp
-L Telemetry-rescue:STM32F303CBx-Misc U101
+P 7350 4500
+F 0 "#PWR0125" H 7350 4350 50  0001 C CNN
+F 1 "+3V3" H 7365 4673 50  0000 C CNN
+F 2 "" H 7350 4500 50  0001 C CNN
+F 3 "" H 7350 4500 50  0001 C CNN
+	1    7350 4500
+	1    0    0    -1
+$EndComp
+Wire Wire Line
+	7350 4500 7350 4600
+Wire Wire Line
+	7350 4600 6950 4600
+$Comp
+L Telemetry-rescue:STM32F303CBx-Misc-Telemetry-rescue U101
 U 1 1 5CE38426
 P 5450 3100
@@
 	1    0    0    -1
 $EndComp
-Text Notes 7200 4500 0    50   ~ 0
+Text Notes 6900 4700 0    50   ~ 0
 ERROR LED
 $Comp
 L Device:R R103
 U 1 1 5CF2EC11
-P 6600 4400
-F 0 "R103" V 6500 4400 50  0000 C CNN
-F 1 "470R" V 6600 4400 50  0000 C CNN
-F 2 "Resistor_SMD:R_0603_1608Metric_Pad1.05x0.95mm_HandSolder" V 6530 4400 50  0001 C CNN
-F 3 "~" H 6600 4400 50  0001 C CNN
-	1    6600 4400
+P 6300 4600
+F 0 "R103" V 6200 4600 50  0000 C CNN
+F 1 "470R" V 6300 4600 50  0000 C CNN
+F 2 "Resistor_SMD:R_0603_1608Metric_Pad1.05x0.95mm_HandSolder" V 6230 4600 50  0001 C CNN
+F 3 "~" H 6300 4600 50  0001 C CNN
+	1    6300 4600
 	0    1    1    0
 $EndComp
 Wire Wire Line
-	6950 4400 6750 4400
-Wire Wire Line
-	6050 4400 6450 4400
+	6650 4600 6450 4600
 $Comp
 L Device:C_Small C106
@@
 	6050 1400 6200 1400
 Wire Wire Line
-	8250 1800 6050 1800
-Wire Wire Line
-	6050 1600 8050 1600
-Wire Wire Line
-	8050 1300 8050 1600
-Wire Wire Line
-	8150 1400 9500 1400
-Wire Wire Line
-	6050 1700 8150 1700
-Wire Wire Line
-	8150 1400 8150 1700
-Wire Wire Line
-	6050 1500 9500 1500
-Wire Wire Line
-	9500 1750 9400 1750
+	9500 1750 9450 1750
 $Comp
 L Mechanical:MountingHole MH101
@@
 Text GLabel 6150 4100 2    50   Output ~ 0
 AMP_CS
-Wire Wire Line
-	6050 4600 6150 4600
 $Comp
 L Connector:TestPoint TP101
@@
 	1800 1850 1800 1900
 $Comp
-L Telemetry-rescue:SG-310_SCF_8.000000MHZ-Misc X101
+L Telemetry-rescue:SG-310_SCF_8.000000MHZ-Misc-Telemetry-rescue X101
 U 1 1 5CECEA0C
 P 3900 2000
@@
 	3450 1650 3900 1650
 Wire Wire Line
-	8050 1300 9500 1300
-Wire Wire Line
 	10400 1500 10400 1750
 $Comp
-L Telemetry-rescue:IS25LP032D-Misc U102
+L Telemetry-rescue:IS25LP032D-Misc-Telemetry-rescue U102
 U 1 1 5CF328C7
 P 9950 1400
@@
 Text GLabel 6150 4200 2    50   Output ~ 0
 AMP_DIN
-NoConn ~ 6050 4500
 NoConn ~ 10350 5200
 NoConn ~ 3550 2000
@@
 Text GLabel 6900 3000 2    50   Output ~ 0
 UART_TX
-Text GLabel 9400 1750 0    50   Input ~ 0
-WP
+Text GLabel 9450 1750 0    50   Input ~ 0
+FLASH_WP
 Text GLabel 6150 3800 2    50   Output ~ 0
-WP
+FLASH_WP
 $Comp
 L Device:R R104
@@
 	1    0    0    -1
 $EndComp
-NoConn ~ 6150 4600
 $Comp
 L power:VCC #PWR0123
@@
 Wire Wire Line
 	6500 5750 6500 6050
+Wire Wire Line
+	6150 4600 6050 4600
+Text GLabel 6200 1800 2    50   Output ~ 0
+FLASH_HOLD
+Text GLabel 9450 1650 0    50   Input ~ 0
+FLASH_HOLD
+Wire Wire Line
+	9450 1650 9500 1650
+Text GLabel 6150 4400 2    50   Output ~ 0
+FLASH_CS
+Text GLabel 9450 1200 0    50   Input ~ 0
+FLASH_CS
+Text GLabel 6200 1500 2    50   Output ~ 0
+FLASH_SCK
+Text GLabel 6200 1700 2    50   Output ~ 0
+FLASH_MOSI
+Text GLabel 6200 1600 2    50   Input ~ 0
+FLASH_MISO
+Text GLabel 9450 1300 0    50   Output ~ 0
+FLASH_MISO
+Text GLabel 9450 1500 0    50   Input ~ 0
+FLASH_SCK
+Text GLabel 9450 1400 0    50   Input ~ 0
+FLASH_MOSI
+Wire Wire Line
+	9450 1200 9500 1200
+Wire Wire Line
+	9450 1300 9500 1300
+Wire Wire Line
+	9450 1400 9500 1400
+Wire Wire Line
+	9500 1500 9450 1500
+Wire Wire Line
+	6050 1500 6200 1500
+Wire Wire Line
+	6200 1600 6050 1600
+Wire Wire Line
+	6050 1700 6200 1700
+Wire Wire Line
+	6200 1800 6050 1800
+NoConn ~ 6050 4500
+Wire Wire Line
+	6150 4400 6050 4400
 $EndSCHEMATC
