File: hw/output.sch (KiCad schematic (older format))
At the start: 33 parts, among them J401 Conn_01x02, J402 Conn_01x02, J403 Conn_01x02, J404 Conn_01x02, J405 Conn_01x02, J406 Conn_01x02, J407 Conn_01x02, J408 Conn_01x02, J409 Conn_02x06_Odd_Even, Q401 IRLML6344TRPBF, Q402 IRLML6344TRPBF, Q403 IRLML6344TRPBF, Q404 IRLZ44N, Q405 IRLML6344TRPBF, Q406 IRLML6344TRPBF, Q407 IRLML6344TRPBF, Q408 IRLZ44N

Commit message: Connections updates
Parts:
- added JP401: Jumper_NC_Small, Pin_Headers:Pin_Header_Angled_1x02, symbol Device:Jumper_NC_Small
- J401, J402, J403, J405, J406, J407, J408: footprint (none) -> Connectors_Phoenix:PhoenixContact_MCV-G_02x3.81mm_Vertical
- J404: footprint (none) -> Inductors_NEOSID:Neosid_Inductor_SM-NE150
- J409: value Conn_02x06_Odd_Even -> SERVO_OUT; footprint (none) -> Pin_Headers:Pin_Header_Angled_2x06
- R401, R402, R403, R404, R405, R406, R407, R408, R409, R410, R411, R412, R413, R414, R415, R416: footprint (none) -> Resistors_SMD:R_0603_HandSoldering
Connections:
- wire segments 92 -> 95
Changed lines of the file:
@@
 F 0 "J404" H 2280 1242 50  0000 L CNN
 F 1 "Conn_01x02" H 2280 1151 50  0000 L CNN
-F 2 "" H 2200 1250 50  0001 C CNN
+F 2 "Inductors_NEOSID:Neosid_Inductor_SM-NE150" H 2200 1250 50  0001 C CNN
 F 3 "~" H 2200 1250 50  0001 C CNN
 	1    2200 1250
@@
 F 0 "R408" H 1591 2054 50  0000 R CNN
 F 1 "10k" H 1591 2145 50  0000 R CNN
-F 2 "" H 1650 2100 50  0001 C CNN
+F 2 "Resistors_SMD:R_0603_HandSoldering" H 1650 2100 50  0001 C CNN
 F 3 "~" H 1650 2100 50  0001 C CNN
 	1    1650 2100
@@
 F 0 "J408" H 2280 3342 50  0000 L CNN
 F 1 "Conn_01x02" H 2280 3251 50  0000 L CNN
-F 2 "" H 2200 3350 50  0001 C CNN
+F 2 "Connectors_Phoenix:PhoenixContact_MCV-G_02x3.81mm_Vertical" H 2200 3350 50  0001 C CNN
 F 3 "~" H 2200 3350 50  0001 C CNN
 	1    2200 3350
@@
 F 0 "R416" H 1591 4154 50  0000 R CNN
 F 1 "10k" H 1591 4245 50  0000 R CNN
-F 2 "" H 1650 4200 50  0001 C CNN
+F 2 "Resistors_SMD:R_0603_HandSoldering" H 1650 4200 50  0001 C CNN
 F 3 "~" H 1650 4200 50  0001 C CNN
 	1    1650 4200
@@
 L power:VCC #PWR0417
 U 1 1 5CEA7FEA
-P 1500 5350
-F 0 "#PWR0417" H 1500 5200 50  0001 C CNN
-F 1 "VCC" H 1517 5523 50  0000 C CNN
-F 2 "" H 1500 5350 50  0001 C CNN
-F 3 "" H 1500 5350 50  0001 C CNN
-	1    1500 5350
-	1    0    0    -1
-$EndComp
-$Comp
-L power:VCC #PWR0418
-U 1 1 5CEA800A
-P 2100 5350
-F 0 "#PWR0418" H 2100 5200 50  0001 C CNN
-F 1 "VCC" H 2117 5523 50  0000 C CNN
-F 2 "" H 2100 5350 50  0001 C CNN
-F 3 "" H 2100 5350 50  0001 C CNN
-	1    2100 5350
+P 1500 4900
+F 0 "#PWR0417" H 1500 4750 50  0001 C CNN
+F 1 "VCC" H 1517 5073 50  0000 C CNN
+F 2 "" H 1500 4900 50  0001 C CNN
+F 3 "" H 1500 4900 50  0001 C CNN
+	1    1500 4900
 	1    0    0    -1
 $EndComp
@@
 	2050 5600 2100 5600
 Wire Wire Line
-	2100 5600 2100 5350
+	2100 5600 2100 5200
 Wire Wire Line
 	2050 5900 2100 5900
@@
 	1550 5600 1500 5600
 Wire Wire Line
-	1500 5600 1500 5350
+	1500 5600 1500 5200
 Wire Wire Line
 	1550 5900 1500 5900
@@
 F 0 "J401" H 4330 1192 50  0000 L CNN
 F 1 "Conn_01x02" H 4330 1101 50  0000 L CNN
-F 2 "" H 4250 1200 50  0001 C CNN
+F 2 "Connectors_Phoenix:PhoenixContact_MCV-G_02x3.81mm_Vertical" H 4250 1200 50  0001 C CNN
 F 3 "~" H 4250 1200 50  0001 C CNN
 	1    4250 1200
@@
 F 0 "R405" H 3641 1954 50  0000 R CNN
 F 1 "R_Small" H 3641 2045 50  0000 R CNN
-F 2 "" H 3700 2000 50  0001 C CNN
+F 2 "Resistors_SMD:R_0603_HandSoldering" H 3700 2000 50  0001 C CNN
 F 3 "~" H 3700 2000 50  0001 C CNN
 	1    3700 2000
@@
 F 0 "R401" V 1154 1800 50  0000 C CNN
 F 1 "10" V 1245 1800 50  0000 C CNN
-F 2 "" H 1350 1800 50  0001 C CNN
+F 2 "Resistors_SMD:R_0603_HandSoldering" H 1350 1800 50  0001 C CNN
 F 3 "~" H 1350 1800 50  0001 C CNN
 	1    1350 1800
@@
 F 0 "R412" V 1154 3900 50  0000 C CNN
 F 1 "10" V 1245 3900 50  0000 C CNN
-F 2 "" H 1350 3900 50  0001 C CNN
+F 2 "Resistors_SMD:R_0603_HandSoldering" H 1350 3900 50  0001 C CNN
 F 3 "~" H 1350 3900 50  0001 C CNN
 	1    1350 3900
@@
 F 0 "R402" V 3354 1800 50  0000 C CNN
 F 1 "10" V 3445 1800 50  0000 C CNN
-F 2 "" H 3550 1800 50  0001 C CNN
+F 2 "Resistors_SMD:R_0603_HandSoldering" H 3550 1800 50  0001 C CNN
 F 3 "~" H 3550 1800 50  0001 C CNN
 	1    3550 1800
@@
 F 0 "J405" H 4330 3092 50  0000 L CNN
 F 1 "Conn_01x02" H 4330 3001 50  0000 L CNN
-F 2 "" H 4250 3100 50  0001 C CNN
+F 2 "Connectors_Phoenix:PhoenixContact_MCV-G_02x3.81mm_Vertical" H 4250 3100 50  0001 C CNN
 F 3 "~" H 4250 3100 50  0001 C CNN
 	1    4250 3100
@@
 F 0 "R413" H 3641 3854 50  0000 R CNN
 F 1 "R_Small" H 3641 3945 50  0000 R CNN
-F 2 "" H 3700 3900 50  0001 C CNN
+F 2 "Resistors_SMD:R_0603_HandSoldering" H 3700 3900 50  0001 C CNN
 F 3 "~" H 3700 3900 50  0001 C CNN
 	1    3700 3900
@@
 F 0 "R409" V 3354 3700 50  0000 C CNN
 F 1 "10" V 3445 3700 50  0000 C CNN
-F 2 "" H 3550 3700 50  0001 C CNN
+F 2 "Resistors_SMD:R_0603_HandSoldering" H 3550 3700 50  0001 C CNN
 F 3 "~" H 3550 3700 50  0001 C CNN
 	1    3550 3700
@@
 F 0 "J402" H 6430 1192 50  0000 L CNN
 F 1 "Conn_01x02" H 6430 1101 50  0000 L CNN
-F 2 "" H 6350 1200 50  0001 C CNN
+F 2 "Connectors_Phoenix:PhoenixContact_MCV-G_02x3.81mm_Vertical" H 6350 1200 50  0001 C CNN
 F 3 "~" H 6350 1200 50  0001 C CNN
 	1    6350 1200
@@
 F 0 "R406" H 5741 1954 50  0000 R CNN
 F 1 "R_Small" H 5741 2045 50  0000 R CNN
-F 2 "" H 5800 2000 50  0001 C CNN
+F 2 "Resistors_SMD:R_0603_HandSoldering" H 5800 2000 50  0001 C CNN
 F 3 "~" H 5800 2000 50  0001 C CNN
 	1    5800 2000
@@
 F 0 "R403" V 5454 1800 50  0000 C CNN
 F 1 "10" V 5545 1800 50  0000 C CNN
-F 2 "" H 5650 1800 50  0001 C CNN
+F 2 "Resistors_SMD:R_0603_HandSoldering" H 5650 1800 50  0001 C CNN
 F 3 "~" H 5650 1800 50  0001 C CNN
 	1    5650 1800
@@
 F 0 "J406" H 6430 3092 50  0000 L CNN
 F 1 "Conn_01x02" H 6430 3001 50  0000 L CNN
-F 2 "" H 6350 3100 50  0001 C CNN
+F 2 "Connectors_Phoenix:PhoenixContact_MCV-G_02x3.81mm_Vertical" H 6350 3100 50  0001 C CNN
 F 3 "~" H 6350 3100 50  0001 C CNN
 	1    6350 3100
@@
 F 0 "R414" H 5741 3854 50  0000 R CNN
 F 1 "R_Small" H 5741 3945 50  0000 R CNN
-F 2 "" H 5800 3900 50  0001 C CNN
+F 2 "Resistors_SMD:R_0603_HandSoldering" H 5800 3900 50  0001 C CNN
 F 3 "~" H 5800 3900 50  0001 C CNN
 	1    5800 3900
@@
 F 0 "R410" V 5454 3700 50  0000 C CNN
 F 1 "10" V 5545 3700 50  0000 C CNN
-F 2 "" H 5650 3700 50  0001 C CNN
+F 2 "Resistors_SMD:R_0603_HandSoldering" H 5650 3700 50  0001 C CNN
 F 3 "~" H 5650 3700 50  0001 C CNN
 	1    5650 3700
@@
 P 1750 5700
 F 0 "J409" H 1800 6117 50  0000 C CNN
-F 1 "Conn_02x06_Odd_Even" H 1800 6026 50  0000 C CNN
-F 2 "" H 1750 5700 50  0001 C CNN
+F 1 "SERVO_OUT" H 1800 6026 50  0000 C CNN
+F 2 "Pin_Headers:Pin_Header_Angled_2x06" H 1750 5700 50  0001 C CNN
 F 3 "~" H 1750 5700 50  0001 C CNN
 	1    1750 5700
@@
 F 0 "J403" H 8480 1192 50  0000 L CNN
 F 1 "Conn_01x02" H 8480 1101 50  0000 L CNN
-F 2 "" H 8400 1200 50  0001 C CNN
+F 2 "Connectors_Phoenix:PhoenixContact_MCV-G_02x3.81mm_Vertical" H 8400 1200 50  0001 C CNN
 F 3 "~" H 8400 1200 50  0001 C CNN
 	1    8400 1200
@@
 F 0 "R407" H 7791 1954 50  0000 R CNN
 F 1 "R_Small" H 7791 2045 50  0000 R CNN
-F 2 "" H 7850 2000 50  0001 C CNN
+F 2 "Resistors_SMD:R_0603_HandSoldering" H 7850 2000 50  0001 C CNN
 F 3 "~" H 7850 2000 50  0001 C CNN
 	1    7850 2000
@@
 F 0 "R404" V 7504 1800 50  0000 C CNN
 F 1 "10" V 7595 1800 50  0000 C CNN
-F 2 "" H 7700 1800 50  0001 C CNN
+F 2 "Resistors_SMD:R_0603_HandSoldering" H 7700 1800 50  0001 C CNN
 F 3 "~" H 7700 1800 50  0001 C CNN
 	1    7700 1800
@@
 F 0 "J407" H 8480 3092 50  0000 L CNN
 F 1 "Conn_01x02" H 8480 3001 50  0000 L CNN
-F 2 "" H 8400 3100 50  0001 C CNN
+F 2 "Connectors_Phoenix:PhoenixContact_MCV-G_02x3.81mm_Vertical" H 8400 3100 50  0001 C CNN
 F 3 "~" H 8400 3100 50  0001 C CNN
 	1    8400 3100
@@
 F 0 "R415" H 7791 3854 50  0000 R CNN
 F 1 "R_Small" H 7791 3945 50  0000 R CNN
-F 2 "" H 7850 3900 50  0001 C CNN
+F 2 "Resistors_SMD:R_0603_HandSoldering" H 7850 3900 50  0001 C CNN
 F 3 "~" H 7850 3900 50  0001 C CNN
 	1    7850 3900
@@
 F 0 "R411" V 7504 3700 50  0000 C CNN
 F 1 "10" V 7595 3700 50  0000 C CNN
-F 2 "" H 7700 3700 50  0001 C CNN
+F 2 "Resistors_SMD:R_0603_HandSoldering" H 7700 3700 50  0001 C CNN
 F 3 "~" H 7700 3700 50  0001 C CNN
 	1    7700 3700
@@
 Wire Wire Line
 	7600 3700 7550 3700
+Wire Wire Line
+	2100 5200 1500 5200
+Connection ~ 1500 5200
+Wire Wire Line
+	1500 4900 1500 4950
+Wire Wire Line
+	1500 5150 1500 5200
+$Comp
+L Device:Jumper_NC_Small JP401
+U 1 1 5CE95F20
+P 1500 5050
+F 0 "JP401" V 1546 5003 50  0000 R CNN
+F 1 "Jumper_NC_Small" V 1455 5003 50  0000 R CNN
+F 2 "Pin_Headers:Pin_Header_Angled_1x02" H 1500 5050 50  0001 C CNN
+F 3 "~" H 1500 5050 50  0001 C CNN
+	1    1500 5050
+	0    -1   -1   0
+$EndComp
 $EndSCHEMATC

Commit message: Layout started, schematic modified for easier layout
Parts:
- J401, J402, J403, J405, J406, J407: footprint Connectors_Phoenix:PhoenixContact_MCV-G_02x3.81mm_Vertical -> Pin_Headers:Pin_Header_Angled_1x02_Pitch2.54mm
- J404: footprint Inductors_NEOSID:Neosid_Inductor_SM-NE150 -> Connectors_Phoenix:PhoenixContact_MCV-G_02x3.81mm_Vertical
- JP401: footprint Pin_Headers:Pin_Header_Angled_1x02 -> Pin_Headers:Pin_Header_Straight_1x02
- Q401, Q402, Q403, Q405, Q406, Q407: footprint digikey-footprints:SOT-23-3 -> TO_SOT_Packages_SMD:SOT-23
- Q404, Q408: footprint Package_TO_SOT_THT:TO-220-3_Vertical -> TO_SOT_Packages_THT:TO-220_Vertical
Changed lines of the file:
@@
 F 0 "J404" H 2280 1242 50  0000 L CNN
 F 1 "Conn_01x02" H 2280 1151 50  0000 L CNN
-F 2 "Inductors_NEOSID:Neosid_Inductor_SM-NE150" H 2200 1250 50  0001 C CNN
+F 2 "Connectors_Phoenix:PhoenixContact_MCV-G_02x3.81mm_Vertical" H 2200 1250 50  0001 C CNN
 F 3 "~" H 2200 1250 50  0001 C CNN
 	1    2200 1250
@@
 F 0 "Q404" H 2105 1846 50  0000 L CNN
 F 1 "IRLZ44N" H 2105 1755 50  0000 L CNN
-F 2 "Package_TO_SOT_THT:TO-220-3_Vertical" H 2150 1725 50  0001 L CIN
+F 2 "TO_SOT_Packages_THT:TO-220_Vertical" H 2150 1725 50  0001 L CIN
 F 3 "http://www.irf.com/product-info/datasheets/data/irlz44n.pdf" H 1900 1800 50  0001 L CNN
 	1    1900 1800
@@
 F 0 "Q408" H 2105 3946 50  0000 L CNN
 F 1 "IRLZ44N" H 2105 3855 50  0000 L CNN
-F 2 "Package_TO_SOT_THT:TO-220-3_Vertical" H 2150 3825 50  0001 L CIN
+F 2 "TO_SOT_Packages_THT:TO-220_Vertical" H 2150 3825 50  0001 L CIN
 F 3 "http://www.irf.com/product-info/datasheets/data/irlz44n.pdf" H 1900 3900 50  0001 L CNN
 	1    1900 3900
@@
 	1550 5700 1450 5700
 Wire Wire Line
-	1450 5700 1450 6000
-Wire Wire Line
-	1550 6000 1450 6000
-Connection ~ 1450 6000
-Wire Wire Line
 	2050 5700 2150 5700
 Wire Wire Line
-	2150 5700 2150 6000
-Wire Wire Line
-	2050 6000 2150 6000
-Connection ~ 2150 6000
-Wire Wire Line
-	1550 5800 1200 5800
-Wire Wire Line
 	1550 5500 1200 5500
 Wire Wire Line
 	2050 5500 2350 5500
-Wire Wire Line
-	2050 5800 2350 5800
 Text GLabel 2350 5500 2    50   Input ~ 0
 SERVO_OUT2
-Text GLabel 2350 5800 2    50   Input ~ 0
+Text GLabel 2350 6000 2    50   Input ~ 0
 SERVO_OUT4
-Text GLabel 1200 5800 0    50   Input ~ 0
+Text GLabel 1200 6000 0    50   Input ~ 0
 SERVO_OUT3
 Text GLabel 1200 5500 0    50   Input ~ 0
@@
 F 0 "Q401" H 4157 1753 60  0000 L CNN
 F 1 "IRLML6344TRPBF" H 4157 1647 60  0000 L CNN
-F 2 "digikey-footprints:SOT-23-3" H 4250 1900 60  0001 L CNN
+F 2 "TO_SOT_Packages_SMD:SOT-23" H 4250 1900 60  0001 L CNN
 F 3 "https://www.infineon.com/dgdl/irlml6344pbf.pdf?fileId=5546d462533600a4015356689c44262c" H 4250 2000 60  0001 L CNN
 F 4 "IRLML6344TRPBFCT-ND" H 4250 2100 60  0001 L CNN "Digi-Key_PN"
@@
 F 0 "J401" H 4330 1192 50  0000 L CNN
 F 1 "Conn_01x02" H 4330 1101 50  0000 L CNN
-F 2 "Connectors_Phoenix:PhoenixContact_MCV-G_02x3.81mm_Vertical" H 4250 1200 50  0001 C CNN
+F 2 "Pin_Headers:Pin_Header_Angled_1x02_Pitch2.54mm" H 4250 1200 50  0001 C CNN
 F 3 "~" H 4250 1200 50  0001 C CNN
 	1    4250 1200
@@
 F 0 "Q405" H 4157 3653 60  0000 L CNN
 F 1 "IRLML6344TRPBF" H 4157 3547 60  0000 L CNN
-F 2 "digikey-footprints:SOT-23-3" H 4250 3800 60  0001 L CNN
+F 2 "TO_SOT_Packages_SMD:SOT-23" H 4250 3800 60  0001 L CNN
 F 3 "https://www.infineon.com/dgdl/irlml6344pbf.pdf?fileId=5546d462533600a4015356689c44262c" H 4250 3900 60  0001 L CNN
 F 4 "IRLML6344TRPBFCT-ND" H 4250 4000 60  0001 L CNN "Digi-Key_PN"
@@
 F 0 "J405" H 4330 3092 50  0000 L CNN
 F 1 "Conn_01x02" H 4330 3001 50  0000 L CNN
-F 2 "Connectors_Phoenix:PhoenixContact_MCV-G_02x3.81mm_Vertical" H 4250 3100 50  0001 C CNN
+F 2 "Pin_Headers:Pin_Header_Angled_1x02_Pitch2.54mm" H 4250 3100 50  0001 C CNN
 F 3 "~" H 4250 3100 50  0001 C CNN
 	1    4250 3100
@@
 F 0 "Q402" H 6257 1753 60  0000 L CNN
 F 1 "IRLML6344TRPBF" H 6257 1647 60  0000 L CNN
-F 2 "digikey-footprints:SOT-23-3" H 6350 1900 60  0001 L CNN
+F 2 "TO_SOT_Packages_SMD:SOT-23" H 6350 1900 60  0001 L CNN
 F 3 "https://www.infineon.com/dgdl/irlml6344pbf.pdf?fileId=5546d462533600a4015356689c44262c" H 6350 2000 60  0001 L CNN
 F 4 "IRLML6344TRPBFCT-ND" H 6350 2100 60  0001 L CNN "Digi-Key_PN"
@@
 F 0 "J402" H 6430 1192 50  0000 L CNN
 F 1 "Conn_01x02" H 6430 1101 50  0000 L CNN
-F 2 "Connectors_Phoenix:PhoenixContact_MCV-G_02x3.81mm_Vertical" H 6350 1200 50  0001 C CNN
+F 2 "Pin_Headers:Pin_Header_Angled_1x02_Pitch2.54mm" H 6350 1200 50  0001 C CNN
 F 3 "~" H 6350 1200 50  0001 C CNN
 	1    6350 1200
@@
 F 0 "Q406" H 6257 3653 60  0000 L CNN
 F 1 "IRLML6344TRPBF" H 6257 3547 60  0000 L CNN
-F 2 "digikey-footprints:SOT-23-3" H 6350 3800 60  0001 L CNN
+F 2 "TO_SOT_Packages_SMD:SOT-23" H 6350 3800 60  0001 L CNN
 F 3 "https://www.infineon.com/dgdl/irlml6344pbf.pdf?fileId=5546d462533600a4015356689c44262c" H 6350 3900 60  0001 L CNN
 F 4 "IRLML6344TRPBFCT-ND" H 6350 4000 60  0001 L CNN "Digi-Key_PN"
@@
 F 0 "J406" H 6430 3092 50  0000 L CNN
 F 1 "Conn_01x02" H 6430 3001 50  0000 L CNN
-F 2 "Connectors_Phoenix:PhoenixContact_MCV-G_02x3.81mm_Vertical" H 6350 3100 50  0001 C CNN
+F 2 "Pin_Headers:Pin_Header_Angled_1x02_Pitch2.54mm" H 6350 3100 50  0001 C CNN
 F 3 "~" H 6350 3100 50  0001 C CNN
 	1    6350 3100
@@
 	1    0    0    -1
 $EndComp
-Wire Wire Line
-	2150 6000 2150 6100
-Wire Wire Line
-	1450 6000 1450 6100
 $Comp
 L dk_Transistors-FETs-MOSFETs-Single:IRLML6344TRPBF Q403
@@
 F 0 "Q403" H 8307 1753 60  0000 L CNN
 F 1 "IRLML6344TRPBF" H 8307 1647 60  0000 L CNN
-F 2 "digikey-footprints:SOT-23-3" H 8400 1900 60  0001 L CNN
+F 2 "TO_SOT_Packages_SMD:SOT-23" H 8400 1900 60  0001 L CNN
 F 3 "https://www.infineon.com/dgdl/irlml6344pbf.pdf?fileId=5546d462533600a4015356689c44262c" H 8400 2000 60  0001 L CNN
 F 4 "IRLML6344TRPBFCT-ND" H 8400 2100 60  0001 L CNN "Digi-Key_PN"
@@
 F 0 "J403" H 8480 1192 50  0000 L CNN
 F 1 "Conn_01x02" H 8480 1101 50  0000 L CNN
-F 2 "Connectors_Phoenix:PhoenixContact_MCV-G_02x3.81mm_Vertical" H 8400 1200 50  0001 C CNN
+F 2 "Pin_Headers:Pin_Header_Angled_1x02_Pitch2.54mm" H 8400 1200 50  0001 C CNN
 F 3 "~" H 8400 1200 50  0001 C CNN
 	1    8400 1200
@@
 F 0 "Q407" H 8307 3653 60  0000 L CNN
 F 1 "IRLML6344TRPBF" H 8307 3547 60  0000 L CNN
-F 2 "digikey-footprints:SOT-23-3" H 8400 3800 60  0001 L CNN
+F 2 "TO_SOT_Packages_SMD:SOT-23" H 8400 3800 60  0001 L CNN
 F 3 "https://www.infineon.com/dgdl/irlml6344pbf.pdf?fileId=5546d462533600a4015356689c44262c" H 8400 3900 60  0001 L CNN
 F 4 "IRLML6344TRPBFCT-ND" H 8400 4000 60  0001 L CNN "Digi-Key_PN"
@@
 F 0 "J407" H 8480 3092 50  0000 L CNN
 F 1 "Conn_01x02" H 8480 3001 50  0000 L CNN
-F 2 "Connectors_Phoenix:PhoenixContact_MCV-G_02x3.81mm_Vertical" H 8400 3100 50  0001 C CNN
+F 2 "Pin_Headers:Pin_Header_Angled_1x02_Pitch2.54mm" H 8400 3100 50  0001 C CNN
 F 3 "~" H 8400 3100 50  0001 C CNN
 	1    8400 3100
@@
 F 0 "JP401" V 1546 5003 50  0000 R CNN
 F 1 "Jumper_NC_Small" V 1455 5003 50  0000 R CNN
-F 2 "Pin_Headers:Pin_Header_Angled_1x02" H 1500 5050 50  0001 C CNN
+F 2 "Pin_Headers:Pin_Header_Straight_1x02" H 1500 5050 50  0001 C CNN
 F 3 "~" H 1500 5050 50  0001 C CNN
 	1    1500 5050
 	0    -1   -1   0
 $EndComp
+Wire Wire Line
+	2150 5700 2150 5800
+Wire Wire Line
+	1450 5700 1450 5800
+Wire Wire Line
+	1550 5800 1450 5800
+Connection ~ 1450 5800
+Wire Wire Line
+	1450 5800 1450 6100
+Wire Wire Line
+	2050 5800 2150 5800
+Connection ~ 2150 5800
+Wire Wire Line
+	2150 5800 2150 6100
+Wire Wire Line
+	2050 6000 2350 6000
+Wire Wire Line
+	1550 6000 1200 6000
 $EndSCHEMATC

Commit message: Layout improvements
Signed-off-by: findersee <aki.kuusela@findersee.fi>
Parts:
- Q401, Q402, Q403, Q405, Q406, Q407: footprint TO_SOT_Packages_SMD:SOT-23 -> digikey-footprints:SOT-23-3
Changed lines of the file:
@@
 F 0 "Q401" H 4157 1753 60  0000 L CNN
 F 1 "IRLML6344TRPBF" H 4157 1647 60  0000 L CNN
-F 2 "TO_SOT_Packages_SMD:SOT-23" H 4250 1900 60  0001 L CNN
+F 2 "digikey-footprints:SOT-23-3" H 4250 1900 60  0001 L CNN
 F 3 "https://www.infineon.com/dgdl/irlml6344pbf.pdf?fileId=5546d462533600a4015356689c44262c" H 4250 2000 60  0001 L CNN
 F 4 "IRLML6344TRPBFCT-ND" H 4250 2100 60  0001 L CNN "Digi-Key_PN"
@@
 F 0 "Q405" H 4157 3653 60  0000 L CNN
 F 1 "IRLML6344TRPBF" H 4157 3547 60  0000 L CNN
-F 2 "TO_SOT_Packages_SMD:SOT-23" H 4250 3800 60  0001 L CNN
+F 2 "digikey-footprints:SOT-23-3" H 4250 3800 60  0001 L CNN
 F 3 "https://www.infineon.com/dgdl/irlml6344pbf.pdf?fileId=5546d462533600a4015356689c44262c" H 4250 3900 60  0001 L CNN
 F 4 "IRLML6344TRPBFCT-ND" H 4250 4000 60  0001 L CNN "Digi-Key_PN"
@@
 F 0 "Q402" H 6257 1753 60  0000 L CNN
 F 1 "IRLML6344TRPBF" H 6257 1647 60  0000 L CNN
-F 2 "TO_SOT_Packages_SMD:SOT-23" H 6350 1900 60  0001 L CNN
+F 2 "digikey-footprints:SOT-23-3" H 6350 1900 60  0001 L CNN
 F 3 "https://www.infineon.com/dgdl/irlml6344pbf.pdf?fileId=5546d462533600a4015356689c44262c" H 6350 2000 60  0001 L CNN
 F 4 "IRLML6344TRPBFCT-ND" H 6350 2100 60  0001 L CNN "Digi-Key_PN"
@@
 F 0 "Q406" H 6257 3653 60  0000 L CNN
 F 1 "IRLML6344TRPBF" H 6257 3547 60  0000 L CNN
-F 2 "TO_SOT_Packages_SMD:SOT-23" H 6350 3800 60  0001 L CNN
+F 2 "digikey-footprints:SOT-23-3" H 6350 3800 60  0001 L CNN
 F 3 "https://www.infineon.com/dgdl/irlml6344pbf.pdf?fileId=5546d462533600a4015356689c44262c" H 6350 3900 60  0001 L CNN
 F 4 "IRLML6344TRPBFCT-ND" H 6350 4000 60  0001 L CNN "Digi-Key_PN"
@@
 F 0 "Q403" H 8307 1753 60  0000 L CNN
 F 1 "IRLML6344TRPBF" H 8307 1647 60  0000 L CNN
-F 2 "TO_SOT_Packages_SMD:SOT-23" H 8400 1900 60  0001 L CNN
+F 2 "digikey-footprints:SOT-23-3" H 8400 1900 60  0001 L CNN
 F 3 "https://www.infineon.com/dgdl/irlml6344pbf.pdf?fileId=5546d462533600a4015356689c44262c" H 8400 2000 60  0001 L CNN
 F 4 "IRLML6344TRPBFCT-ND" H 8400 2100 60  0001 L CNN "Digi-Key_PN"
@@
 F 0 "Q407" H 8307 3653 60  0000 L CNN
 F 1 "IRLML6344TRPBF" H 8307 3547 60  0000 L CNN
-F 2 "TO_SOT_Packages_SMD:SOT-23" H 8400 3800 60  0001 L CNN
+F 2 "digikey-footprints:SOT-23-3" H 8400 3800 60  0001 L CNN
 F 3 "https://www.infineon.com/dgdl/irlml6344pbf.pdf?fileId=5546d462533600a4015356689c44262c" H 8400 3900 60  0001 L CNN
 F 4 "IRLML6344TRPBFCT-ND" H 8400 4000 60  0001 L CNN "Digi-Key_PN"

Commit message: Switched High Current FETs and added drivers for those
Parts:
- removed Q404, Q408: IRLZ44N, TO_SOT_Packages_THT:TO-220_Vertical, symbol Transistor_FET:IRLZ44N
- removed R401, R412: 10, Resistors_SMD:R_0603_HandSoldering, symbol Device:R_Small
- removed R408, R416: 10k, Resistors_SMD:R_0603_HandSoldering, symbol Device:R_Small
- added C401, C402: 1u, Capacitors_SMD:C_0805_HandSoldering, symbol Device:C_Small
- added Q404, Q408: CSD17306Q5A, TO_SOT_Packages_SMD:TDSON-8-1_HandSoldering, symbol Transistor_FET:CSD17306Q5A
- added U401, U402: MCP1416, TO_SOT_Packages_SMD:SOT-23-5_HandSoldering, symbol Driver_FET:MCP1416
- J409: footprint Pin_Headers:Pin_Header_Angled_2x06 -> Pin_Headers:Pin_Header_Straight_2x06
Connections:
- wire segments 95 -> 107

Commit message: Lots and lots of updates Added DAC amplifier that can be controlled Cleaned up the schematic
Parts:
- added C403, C405, C406: 100n, Capacitors_SMD:C_0603_HandSoldering, symbol Device:C_Small
- added C404: 10u, Capacitors_SMD:C_0603_HandSoldering, symbol Device:C_Small
- added J410: AUDIO, Pin_Headers:Pin_Header_Straight_1x02_Pitch2.54mm, symbol Connector_Generic:Conn_01x02
- added R401, R408: 10k, Resistors_SMD:R_0603_HandSoldering, symbol Device:R_Small
- added U403: MCP4012-xxxxCH, TO_SOT_Packages_SMD:SOT-23-6_Handsoldering, symbol Potentiometer_Digital:MCP4012-xxxxCH
- added U404: OP179GRT, TO_SOT_Packages_SMD:SOT-23-5_HandSoldering, symbol Amplifier_Operational:OP179GRT
Connections:
- net labels added: +5VA, AMP_CS, AMP_DIR, DAC_OUT
- wire segments 107 -> 143
Other:
- note added: "DAC AMPLIFIER"
- note added: "HIGH CURRENT PWM OUTPUTS"
- note added: "ON/OFF OUTPUTS"
- note added: "PWM OUTPUTS"
- note added: "SERVO OUTPUTS"

Commit message: Added SWD connector for debugging
Parts:
- removed U404: OP179GRT, TO_SOT_Packages_SMD:SOT-23-5_HandSoldering, symbol Amplifier_Operational:OP179GRT
- added U404: MCP6001-OT, Package_TO_SOT_SMD:SOT-23-5, symbol Amplifier_Operational:MCP6001-OT
Changed lines of the file:
@@
-$EndComp
-$Comp
-L Amplifier_Operational:OP179GRT U404
-U 1 1 5CEBD0B8
-P 5100 7150
-F 0 "U404" H 5100 7300 50  0000 L CNN
-F 1 "OP179GRT" H 5050 6950 50  0000 L CNN
-F 2 "TO_SOT_Packages_SMD:SOT-23-5_HandSoldering" H 5100 7150 50  0001 C CNN
-F 3 "http://www.analog.com/media/en/technical-documentation/data-sheets/OP179_279.pdf" H 5100 7350 50  0001 C CNN
-	1    5100 7150
-	1    0    0    -1
 $EndComp
 $Comp
@@
 Text Notes 600  5500 0    50   ~ 0
 SERVO OUTPUTS
+$Comp
+L Amplifier_Operational:MCP6001-OT U404
+U 1 1 5CEC9F24
+P 5100 7150
+F 0 "U404" H 5100 7300 50  0000 L CNN
+F 1 "MCP6001-OT" H 5100 7000 50  0001 L CNN
+F 2 "Package_TO_SOT_SMD:SOT-23-5" H 5000 6950 50  0001 L CNN
+F 3 "http://ww1.microchip.com/downloads/en/DeviceDoc/21733j.pdf" H 5100 7350 50  0001 C CNN
+	1    5100 7150
+	1    0    0    -1
+$EndComp
 $EndSCHEMATC

Commit message: Changed the digital potentiometer to AD5160 10k version and enabled SPI3
Parts:
- removed U403: MCP4012-xxxxCH, TO_SOT_Packages_SMD:SOT-23-6_Handsoldering, symbol Potentiometer_Digital:MCP4012-xxxxCH
- added R412: 0R, Resistors_SMD:R_0402_NoSilk, symbol Device:R_Small
- added U403: AD5160BRJZ10-R2, digikey-footprints:SOT-23-8, symbol Misc:AD5160BRJZ10-R2
- U404: footprint Package_TO_SOT_SMD:SOT-23-5 -> TO_SOT_Packages_SMD:SOT-23-5_HandSoldering
Connections:
- net labels added: AMP_CLK, AMP_DIN
- net labels removed: AMP_DIR
- wire segments 143 -> 151
Other:
- moved on the sheet: Q408

Commit message: Refactored schematic net names
Connections:
- net labels added: SERVO_1, SERVO_2, SERVO_3, SERVO_4
- net labels removed: SERVO_OUT1, SERVO_OUT2, SERVO_OUT3, SERVO_OUT4
Changed lines of the file:
@@
 	2100 6400 2400 6400
 Text GLabel 2400 6400 2    50   Input ~ 0
-SERVO_OUT2
+SERVO_2
 Text GLabel 2400 6900 2    50   Input ~ 0
-SERVO_OUT4
+SERVO_4
 Text GLabel 1250 6900 0    50   Input ~ 0
-SERVO_OUT3
+SERVO_3
 Text GLabel 1250 6400 0    50   Input ~ 0
-SERVO_OUT1
+SERVO_1
 $Comp
 L dk_Transistors-FETs-MOSFETs-Single:IRLML6344TRPBF Q401
