File: hw/output.sch (KiCad schematic (older format))
At the start: 44 parts, among them J401 Conn_01x02, J402 Conn_01x02, J403 Conn_01x02, J404 Conn_01x02, J405 Conn_01x02, J406 Conn_01x02, J407 Conn_01x02, J408 Conn_01x02, J409 SERVO_OUT, J410 AUDIO, Q401 IRLML6344TRPBF, Q402 IRLML6344TRPBF, Q403 IRLML6344TRPBF, Q404 CSD17306Q5A, Q406 IRLML6344TRPBF, Q408 CSD17306Q5A, U401 MCP1416, U402 MCP1416, U403 AD5160BRJZ10-R2, U404 MCP6001-OT, U405 TLP2361_TPL_E, U406 TLP2361_TPL_E

Commit message: Updates to board revision 0.2 and newer HAL version
Parts:
- removed J409: SERVO_OUT, Pin_Headers:Pin_Header_Straight_2x06, symbol Connector_Generic:Conn_02x06_Odd_Even
- added J409: ServoCon, Connector_PinHeader_2.54mm:PinHeader_2x03_P2.54mm_Vertical, symbol Connector_Generic:Conn_02x03_Odd_Even
- U401, U402: symbol Driver_FET:MCP1416 -> Telemetry-rescue:MCP1416-Driver_FET
- U403: symbol Misc:AD5160BRJZ10-R2 -> Telemetry-rescue:AD5160BRJZ10-R2-Misc
Connections:
- net labels removed: SERVO_3, SERVO_4
- wire segments 157 -> 147
Changed lines of the file:
@@
 EESchema Schematic File Version 4
-LIBS:Telemetry-cache
-EELAYER 26 0
+EELAYER 30 0
 EELAYER END
 $Descr A4 11693 8268
@@
 Sheet 4 4
 Title "RC Telemetry board"
-Date "2019-05-20"
-Rev "0.1"
+Date "2020-02-12"
+Rev "0.2"
 Comp "www.findersee.fi"
-Comment1 ""
+Comment1 "https://github.com/findersee/rctelemetry"
 Comment2 ""
 Comment3 ""
@@
 	2150 6500 2150 6100
 Wire Wire Line
-	2100 6800 2150 6800
-Wire Wire Line
-	2150 6800 2150 6500
-Connection ~ 2150 6500
-Wire Wire Line
 	1600 6500 1550 6500
 Wire Wire Line
 	1550 6500 1550 6100
-Wire Wire Line
-	1600 6800 1550 6800
-Wire Wire Line
-	1550 6800 1550 6500
-Connection ~ 1550 6500
 Wire Wire Line
 	1600 6600 1500 6600
@@
 Text GLabel 2400 6400 2    50   Input ~ 0
 SERVO_2
-Text GLabel 2400 6900 2    50   Input ~ 0
-SERVO_4
-Text GLabel 1250 6900 0    50   Input ~ 0
-SERVO_3
 Text GLabel 1250 6400 0    50   Input ~ 0
 SERVO_1
@@
 	4900 3650 4850 3650
 $Comp
-L Connector_Generic:Conn_02x06_Odd_Even J409
-U 1 1 5CEF71B9
-P 1800 6600
-F 0 "J409" H 1850 7017 50  0000 C CNN
-F 1 "SERVO_OUT" H 1850 6926 50  0000 C CNN
-F 2 "Pin_Headers:Pin_Header_Straight_2x06" H 1800 6600 50  0001 C CNN
-F 3 "~" H 1800 6600 50  0001 C CNN
-	1    1800 6600
-	1    0    0    -1
-$EndComp
-$Comp
 L power:VCC #PWR0404
 U 1 1 5CEFB1E7
@@
 	0    -1   -1   0
 $EndComp
-Wire Wire Line
-	2200 6600 2200 6700
-Wire Wire Line
-	1500 6600 1500 6700
-Wire Wire Line
-	1600 6700 1500 6700
-Connection ~ 1500 6700
-Wire Wire Line
-	1500 6700 1500 7000
-Wire Wire Line
-	2100 6700 2200 6700
-Connection ~ 2200 6700
-Wire Wire Line
-	2200 6700 2200 7000
-Wire Wire Line
-	2100 6900 2400 6900
-Wire Wire Line
-	1600 6900 1250 6900
-$Comp
-L Driver_FET:MCP1416 U402
+$Comp
+L Telemetry-rescue:MCP1416-Driver_FET U402
 U 1 1 5CEC7B81
 P 1650 3650
+AR Path="/5CEC7B81" Ref="U402"  Part="1"
+AR Path="/5CEA3FFC/5CEC7B81" Ref="U402"  Part="1"
 F 0 "U402" H 1750 3900 50  0000 L CNN
 F 1 "MCP1416" H 1750 3400 50  0000 L CNN
@@
 	2700 2950 2700 3100
 $Comp
-L Driver_FET:MCP1416 U401
+L Telemetry-rescue:MCP1416-Driver_FET U401
 U 1 1 5CED0BC8
 P 1700 1800
+AR Path="/5CED0BC8" Ref="U401"  Part="1"
+AR Path="/5CEA3FFC/5CED0BC8" Ref="U401"  Part="1"
 F 0 "U401" H 1800 2050 50  0000 L CNN
 F 1 "MCP1416" H 1800 1550 50  0000 L CNN
@@
 	4700 6050 4750 6050
 $Comp
-L Misc:AD5160BRJZ10-R2 U403
+L Telemetry-rescue:AD5160BRJZ10-R2-Misc U403
 U 1 1 5CEF134B
 P 4100 6100
@@
 Wire Wire Line
 	10100 2000 10100 2100
+$Comp
+L Connector_Generic:Conn_02x03_Odd_Even J409
+U 1 1 5E5305C4
+P 1800 6500
+F 0 "J409" H 1850 6817 50  0000 C CNN
+F 1 "ServoCon" H 1850 6726 50  0000 C CNN
+F 2 "Connector_PinHeader_2.54mm:PinHeader_2x03_P2.54mm_Vertical" H 1800 6500 50  0001 C CNN
+F 3 "~" H 1800 6500 50  0001 C CNN
+	1    1800 6500
+	1    0    0    -1
+$EndComp
+Wire Wire Line
+	1500 6600 1500 7000
+Wire Wire Line
+	2200 6600 2200 7000
 $EndSCHEMATC

Commit message: Pin remapping and layout improvements
Parts:
- C401, C402: footprint Capacitors_SMD:C_0805_HandSoldering -> Capacitor_SMD:C_0805_2012Metric_Pad1.15x1.40mm_HandSolder
- C403, C404, C405, C406, C407, C408: footprint Capacitors_SMD:C_0603_HandSoldering -> Capacitor_SMD:C_0603_1608Metric_Pad1.05x0.95mm_HandSolder
- R401, R402, R403, R404, R405, R406, R407, R408, R409, R410, R411, R414: footprint Resistors_SMD:R_0603_HandSoldering -> Resistor_SMD:R_0603_1608Metric_Pad1.05x0.95mm_HandSolder

Commit message: Changed High current pwm connectors to 5mm pitch versions
Parts:
- J401, J402, J403, J405, J406, J407: footprint Pin_Headers:Pin_Header_Angled_1x02_Pitch2.54mm -> Connector_Molex:Molex_KK-254_AE-6410-02A_1x02_P2.54mm_Vertical
- J404, J408: footprint Connectors_Phoenix:PhoenixContact_MCV-G_02x3.81mm_Vertical -> TerminalBlock_Phoenix:TerminalBlock_Phoenix_PT-1,5-2-5.0-H_1x02_P5.00mm_Horizontal
- J410: footprint Pin_Headers:Pin_Header_Straight_1x02_Pitch2.54mm -> Connector_PinHeader_2.54mm:PinHeader_1x02_P2.54mm_Vertical
- JP401: footprint Pin_Headers:Pin_Header_Straight_1x02 -> Connector_PinHeader_2.54mm:PinHeader_1x02_P2.54mm_Vertical
Changed lines of the file:
@@
 F 0 "J404" H 2980 1242 50  0000 L CNN
 F 1 "Conn_01x02" H 2980 1151 50  0000 L CNN
-F 2 "Connectors_Phoenix:PhoenixContact_MCV-G_02x3.81mm_Vertical" H 2900 1250 50  0001 C CNN
+F 2 "TerminalBlock_Phoenix:TerminalBlock_Phoenix_PT-1,5-2-5.0-H_1x02_P5.00mm_Horizontal" H 2900 1250 50  0001 C CNN
 F 3 "~" H 2900 1250 50  0001 C CNN
 	1    2900 1250
@@
 F 0 "J408" H 2980 3092 50  0000 L CNN
 F 1 "Conn_01x02" H 2980 3001 50  0000 L CNN
-F 2 "Connectors_Phoenix:PhoenixContact_MCV-G_02x3.81mm_Vertical" H 2900 3100 50  0001 C CNN
+F 2 "TerminalBlock_Phoenix:TerminalBlock_Phoenix_PT-1,5-2-5.0-H_1x02_P5.00mm_Horizontal" H 2900 3100 50  0001 C CNN
 F 3 "~" H 2900 3100 50  0001 C CNN
 	1    2900 3100
@@
 F 0 "J401" H 5780 1192 50  0000 L CNN
 F 1 "Conn_01x02" H 5780 1101 50  0000 L CNN
-F 2 "Pin_Headers:Pin_Header_Angled_1x02_Pitch2.54mm" H 5700 1200 50  0001 C CNN
+F 2 "Connector_Molex:Molex_KK-254_AE-6410-02A_1x02_P2.54mm_Vertical" H 5700 1200 50  0001 C CNN
 F 3 "~" H 5700 1200 50  0001 C CNN
 	1    5700 1200
@@
 F 0 "J405" H 9230 1692 50  0000 L CNN
 F 1 "Conn_01x02" H 9230 1601 50  0000 L CNN
-F 2 "Pin_Headers:Pin_Header_Angled_1x02_Pitch2.54mm" H 9150 1700 50  0001 C CNN
+F 2 "Connector_Molex:Molex_KK-254_AE-6410-02A_1x02_P2.54mm_Vertical" H 9150 1700 50  0001 C CNN
 F 3 "~" H 9150 1700 50  0001 C CNN
 	1    9150 1700
@@
 F 0 "J402" H 7880 1192 50  0000 L CNN
 F 1 "Conn_01x02" H 7880 1101 50  0000 L CNN
-F 2 "Pin_Headers:Pin_Header_Angled_1x02_Pitch2.54mm" H 7800 1200 50  0001 C CNN
+F 2 "Connector_Molex:Molex_KK-254_AE-6410-02A_1x02_P2.54mm_Vertical" H 7800 1200 50  0001 C CNN
 F 3 "~" H 7800 1200 50  0001 C CNN
 	1    7800 1200
@@
 F 0 "J406" H 5780 3042 50  0000 L CNN
 F 1 "Conn_01x02" H 5780 2951 50  0000 L CNN
-F 2 "Pin_Headers:Pin_Header_Angled_1x02_Pitch2.54mm" H 5700 3050 50  0001 C CNN
+F 2 "Connector_Molex:Molex_KK-254_AE-6410-02A_1x02_P2.54mm_Vertical" H 5700 3050 50  0001 C CNN
 F 3 "~" H 5700 3050 50  0001 C CNN
 	1    5700 3050
@@
 F 0 "J403" H 7880 3042 50  0000 L CNN
 F 1 "Conn_01x02" H 7880 2951 50  0000 L CNN
-F 2 "Pin_Headers:Pin_Header_Angled_1x02_Pitch2.54mm" H 7800 3050 50  0001 C CNN
+F 2 "Connector_Molex:Molex_KK-254_AE-6410-02A_1x02_P2.54mm_Vertical" H 7800 3050 50  0001 C CNN
 F 3 "~" H 7800 3050 50  0001 C CNN
 	1    7800 3050
@@
 F 0 "J407" H 9230 3392 50  0000 L CNN
 F 1 "Conn_01x02" H 9230 3301 50  0000 L CNN
-F 2 "Pin_Headers:Pin_Header_Angled_1x02_Pitch2.54mm" H 9150 3400 50  0001 C CNN
+F 2 "Connector_Molex:Molex_KK-254_AE-6410-02A_1x02_P2.54mm_Vertical" H 9150 3400 50  0001 C CNN
 F 3 "~" H 9150 3400 50  0001 C CNN
 	1    9150 3400
@@
 F 0 "JP401" V 1596 5903 50  0000 R CNN
 F 1 "Jumper_NC_Small" V 1505 5903 50  0000 R CNN
-F 2 "Pin_Headers:Pin_Header_Straight_1x02" H 1550 5950 50  0001 C CNN
+F 2 "Connector_PinHeader_2.54mm:PinHeader_1x02_P2.54mm_Vertical" H 1550 5950 50  0001 C CNN
 F 3 "~" H 1550 5950 50  0001 C CNN
 	1    1550 5950
@@
 F 0 "J410" H 6420 6925 50  0000 C CNN
 F 1 "AUDIO" H 6420 7016 50  0000 C CNN
-F 2 "Pin_Headers:Pin_Header_Straight_1x02_Pitch2.54mm" H 6500 7250 50  0001 C CNN
+F 2 "Connector_PinHeader_2.54mm:PinHeader_1x02_P2.54mm_Vertical" H 6500 7250 50  0001 C CNN
 F 3 "~" H 6500 7250 50  0001 C CNN
 	1    6500 7250
