File: hw/Power.sch (KiCad schematic (older format))
At the start: 22 parts

Commit message: Updated pin assignments and preliminary timer2 setup
Signed-off-by: findersee <aki.kuusela@findersee.fi>
Parts:
- removed R?: N/A, symbol Device:R
- removed R?: 0R, symbol Device:R
- gave numbers to parts that had none: 20
Connections:
- wire segments 73 -> 67

Commit message: Connections updates
Parts:
- removed F201: Fuse, symbol Device:Fuse
- added C207: 100n, Capacitors_SMD:C_0805, symbol Device:C
- added C208: 22u, Capacitors_ThroughHole:C_Radial_D7.5_L11.2_P2.5, symbol Device:CP
- added D202: D_Schottky, Diodes_SMD:D_SMA_Handsoldering, symbol Device:D_Schottky
- added D?: D_Schottky, Diodes_SMD:D_SOD-123, symbol Device:D_Schottky
- added L202: 47u, Inductors_NEOSID:Neosid_Inductor_SM-NE127, symbol pspice:INDUCTOR
- added Q201: AO3401A, digikey-footprints:SOT-23-3, symbol dk_Transistors-FETs-MOSFETs-Single:AO3401A
- added R209: R_Small, Resistors_SMD:R_0603_HandSoldering, symbol Device:R_Small
- C201, C202: value CP -> 22u; footprint (none) -> Capacitors_ThroughHole:C_Radial_D7.5_L11.2_P2.5
- C203: footprint (none) -> Capacitors_SMD:C_0603_HandSoldering
- C204: value CP -> 22u
- C205: value C -> 1u; footprint (none) -> Capacitors_SMD:C_0805
- C206: value C -> 2u2; footprint (none) -> Capacitors_SMD:C_0805
- D201: footprint (none) -> Diodes_SMD:D_SOD-123
- J201: footprint (none) -> Connect:JWT_Vertical_A3963-RM3.96mm-2
- L201: footprint (none) -> Inductors_NEOSID:Neosid_Inductor_SM-NE56_SMD2220
- R201, R202, R204, R206, R207, R208: footprint (none) -> Resistors_SMD:R_0603_HandSoldering
- R203: value 75k -> 68k; footprint (none) -> Resistors_SMD:R_0603_HandSoldering
- R205: value 75k -> 12k; footprint (none) -> Resistors_SMD:R_0603_HandSoldering
- U201: footprint (none) -> TO_SOT_Packages_SMD:TO-263-5_TabPin3
- U202: footprint (none) -> TO_SOT_Packages_SMD:SOT-23-6_Handsoldering
Connections:
- wire segments 67 -> 86

Commit message: Layout started, schematic modified for easier layout
Parts:
- C204: footprint (none) -> Capacitors_SMD:C_0805
- J201: footprint Connect:JWT_Vertical_A3963-RM3.96mm-2 -> PCBDecals:2Pin_4mm
- Q201: footprint digikey-footprints:SOT-23-3 -> TO_SOT_Packages_SMD:SOT-23
- gave numbers to parts that had none: 1
Changed lines of the file:
@@
 F 0 "J201" H 920 1275 50  0000 C CNN
 F 1 "Conn_01x02" H 920 1366 50  0000 C CNN
-F 2 "Connect:JWT_Vertical_A3963-RM3.96mm-2" H 1000 1600 50  0001 C CNN
+F 2 "PCBDecals:2Pin_4mm" H 1000 1600 50  0001 C CNN
 F 3 "~" H 1000 1600 50  0001 C CNN
 	1    1000 1600
@@
 F 0 "C204" H 1618 3896 50  0000 L CNN
 F 1 "22u" H 1618 3805 50  0000 L CNN
-F 2 "" H 1538 3700 50  0001 C CNN
+F 2 "Capacitors_SMD:C_0805" H 1538 3700 50  0001 C CNN
 F 3 "~" H 1500 3850 50  0001 C CNN
 	1    1500 3850
@@
 F 0 "Q201" V 2467 2700 60  0000 C CNN
 F 1 "AO3401A" V 2361 2700 60  0000 C CNN
-F 2 "digikey-footprints:SOT-23-3" H 2400 2900 60  0001 L CNN
+F 2 "TO_SOT_Packages_SMD:SOT-23" H 2400 2900 60  0001 L CNN
 F 3 "http://aosmd.com/res/data_sheets/AO3401A.pdf" H 2400 3000 60  0001 L CNN
 F 4 "785-1001-1-ND" H 2400 3100 60  0001 L CNN "Digi-Key_PN"
@@
 	4400 1950 4400 2000
 $Comp
-L Device:D_Schottky D?
+L Device:D_Schottky D203
 U 1 1 5CF6D61D
 P 1150 3650
-F 0 "D?" V 1104 3729 50  0000 L CNN
+F 0 "D203" V 1104 3729 50  0000 L CNN
 F 1 "D_Schottky" V 1195 3729 50  0000 L CNN
 F 2 "Diodes_SMD:D_SOD-123" H 1150 3650 50  0001 C CNN

Commit message: Layout improvements
Signed-off-by: findersee <aki.kuusela@findersee.fi>
Parts:
- removed C207: 100n, Capacitors_SMD:C_0805, symbol Device:C
- removed D203: D_Schottky, Diodes_SMD:D_SOD-123, symbol Device:D_Schottky
- added Q202: AO3401A, digikey-footprints:SOT-23-3, symbol dk_Transistors-FETs-MOSFETs-Single:AO3401A
- added Q203, Q204: IRLML6344TRPBF, digikey-footprints:SOT-23-3, symbol dk_Transistors-FETs-MOSFETs-Single:IRLML6344TRPBF
- added R210, R212, R214: 100k, Resistors_SMD:R_0603_HandSoldering, symbol Device:R_Small
- added R211, R213: 10k, Resistors_SMD:R_0603_HandSoldering, symbol Device:R_Small
- C204: footprint Capacitors_SMD:C_0805 -> Capacitors_ThroughHole:C_Radial_D7.5_L11.2_P2.5
- Q201: footprint TO_SOT_Packages_SMD:SOT-23 -> digikey-footprints:SOT-23-3
- R209: value R_Small -> 100k
Connections:
- net labels added: VBUS
- wire segments 86 -> 114

Commit message: Lots and lots of updates Added DAC amplifier that can be controlled Cleaned up the schematic
Parts:
- L201: footprint Inductors_NEOSID:Neosid_Inductor_SM-NE56_SMD2220 -> Inductors:Inductor_Taiyo-Yuden_MD-3030
- L202: footprint Inductors_NEOSID:Neosid_Inductor_SM-NE127 -> PCBDecals:12x12_inductor
Changed lines of the file:
@@
 F 0 "L201" V 4240 4600 50  0000 C CNN
 F 1 "4u7" V 4149 4600 50  0000 C CNN
-F 2 "Inductors_NEOSID:Neosid_Inductor_SM-NE56_SMD2220" H 4050 4600 50  0001 C CNN
+F 2 "Inductors:Inductor_Taiyo-Yuden_MD-3030" H 4050 4600 50  0001 C CNN
 F 3 "~" H 4050 4600 50  0001 C CNN
 	1    4050 4600
@@
 F 0 "L202" H 5000 2065 50  0000 C CNN
 F 1 "47u" H 5000 1974 50  0000 C CNN
-F 2 "Inductors_NEOSID:Neosid_Inductor_SM-NE127" H 5000 1850 50  0001 C CNN
+F 2 "PCBDecals:12x12_inductor" H 5000 1850 50  0001 C CNN
 F 3 "" H 5000 1850 50  0001 C CNN
 	1    5000 1850

Commit message: Added SWD connector for debugging
Parts:
- D201: footprint Diodes_SMD:D_SOD-123 -> Diodes_SMD:D_SMA_Handsoldering

Commit message: Renamed schematic pdf Added gerbers Added layout pdf Fixed silkscreen on layout
Parts:
- D201, D202: value D_Schottky -> SS54
- L201: value 4u7 -> SPN30304R7MPTE; LCSC Part-number (none) -> C359291
- L202: value 47u -> BCRH1212Y-680M; LCSC Part-number (none) -> C238002
