File: hw/current.sch (KiCad schematic (older format))
At the start: 19 parts

Commit message: Updated pin assignments and preliminary timer2 setup
Signed-off-by: findersee <aki.kuusela@findersee.fi>
Parts:
- gave numbers to parts that had none: 19

Commit message: Connections updates
Parts:
- C301: footprint (none) -> Capacitors_SMD:C_0603
- C302: footprint (none) -> Capacitors_SMD:C_0805
- C303, C305, C306, C307, C308: value C_Small -> 100n; footprint (none) -> Capacitors_SMD:C_0603_HandSoldering
- C304: footprint (none) -> Capacitors_SMD:C_0603_HandSoldering
- J301, J302: footprint (none) -> Connectors_Phoenix:PhoenixContact_MCV-G_02x3.81mm_Vertical
- R301, R303: value R_Small -> 68k; footprint (none) -> Resistors_SMD:R_0603_HandSoldering
- R302, R304: value R_Small -> 12k; footprint (none) -> Resistors_SMD:R_0603_HandSoldering
Changed lines of the file:
@@
 F 0 "J301" H 7180 2742 50  0000 L CNN
 F 1 "Conn_01x02" H 7180 2651 50  0000 L CNN
-F 2 "" H 7100 2750 50  0001 C CNN
+F 2 "Connectors_Phoenix:PhoenixContact_MCV-G_02x3.81mm_Vertical" H 7100 2750 50  0001 C CNN
 F 3 "~" H 7100 2750 50  0001 C CNN
 	1    7100 2750
@@
 F 0 "J302" H 7180 5042 50  0000 L CNN
 F 1 "Conn_01x02" H 7180 4951 50  0000 L CNN
-F 2 "" H 7100 5050 50  0001 C CNN
+F 2 "Connectors_Phoenix:PhoenixContact_MCV-G_02x3.81mm_Vertical" H 7100 5050 50  0001 C CNN
 F 3 "~" H 7100 5050 50  0001 C CNN
 	1    7100 5050
@@
 P 6650 3000
 F 0 "R301" H 6709 3046 50  0000 L CNN
-F 1 "R_Small" H 6709 2955 50  0000 L CNN
-F 2 "" H 6650 3000 50  0001 C CNN
+F 1 "68k" H 6709 2955 50  0000 L CNN
+F 2 "Resistors_SMD:R_0603_HandSoldering" H 6650 3000 50  0001 C CNN
 F 3 "~" H 6650 3000 50  0001 C CNN
 	1    6650 3000
@@
 P 6650 3300
 F 0 "R302" H 6709 3346 50  0000 L CNN
-F 1 "R_Small" H 6709 3255 50  0000 L CNN
-F 2 "" H 6650 3300 50  0001 C CNN
+F 1 "12k" H 6709 3255 50  0000 L CNN
+F 2 "Resistors_SMD:R_0603_HandSoldering" H 6650 3300 50  0001 C CNN
 F 3 "~" H 6650 3300 50  0001 C CNN
 	1    6650 3300
@@
 P 6850 3300
 F 0 "C305" H 6758 3254 50  0000 R CNN
-F 1 "C_Small" H 6758 3345 50  0000 R CNN
-F 2 "" H 6850 3300 50  0001 C CNN
+F 1 "100n" H 6758 3345 50  0000 R CNN
+F 2 "Capacitors_SMD:C_0603_HandSoldering" H 6850 3300 50  0001 C CNN
 F 3 "~" H 6850 3300 50  0001 C CNN
 	1    6850 3300
@@
 P 6650 5300
 F 0 "R303" H 6709 5346 50  0000 L CNN
-F 1 "R_Small" H 6709 5255 50  0000 L CNN
-F 2 "" H 6650 5300 50  0001 C CNN
+F 1 "68k" H 6709 5255 50  0000 L CNN
+F 2 "Resistors_SMD:R_0603_HandSoldering" H 6650 5300 50  0001 C CNN
 F 3 "~" H 6650 5300 50  0001 C CNN
 	1    6650 5300
@@
 P 6650 5600
 F 0 "R304" H 6709 5646 50  0000 L CNN
-F 1 "R_Small" H 6709 5555 50  0000 L CNN
-F 2 "" H 6650 5600 50  0001 C CNN
+F 1 "12k" H 6709 5555 50  0000 L CNN
+F 2 "Resistors_SMD:R_0603_HandSoldering" H 6650 5600 50  0001 C CNN
 F 3 "~" H 6650 5600 50  0001 C CNN
 	1    6650 5600
@@
 P 6850 5600
 F 0 "C308" H 6758 5554 50  0000 R CNN
-F 1 "C_Small" H 6758 5645 50  0000 R CNN
-F 2 "" H 6850 5600 50  0001 C CNN
+F 1 "100n" H 6758 5645 50  0000 R CNN
+F 2 "Capacitors_SMD:C_0603_HandSoldering" H 6850 5600 50  0001 C CNN
 F 3 "~" H 6850 5600 50  0001 C CNN
 	1    6850 5600
@@
 P 7000 1750
 F 0 "C303" V 6771 1750 50  0000 C CNN
-F 1 "C_Small" V 6862 1750 50  0000 C CNN
-F 2 "" H 7000 1750 50  0001 C CNN
+F 1 "100n" V 6862 1750 50  0000 C CNN
+F 2 "Capacitors_SMD:C_0603_HandSoldering" H 7000 1750 50  0001 C CNN
 F 3 "~" H 7000 1750 50  0001 C CNN
 	1    7000 1750
@@
 P 6850 4000
 F 0 "C306" V 6621 4000 50  0000 C CNN
-F 1 "C_Small" V 6712 4000 50  0000 C CNN
-F 2 "" H 6850 4000 50  0001 C CNN
+F 1 "100n" V 6712 4000 50  0000 C CNN
+F 2 "Capacitors_SMD:C_0603_HandSoldering" H 6850 4000 50  0001 C CNN
 F 3 "~" H 6850 4000 50  0001 C CNN
 	1    6850 4000
@@
 P 8000 5200
 F 0 "C307" V 7771 5200 50  0000 C CNN
-F 1 "C_Small" V 7862 5200 50  0000 C CNN
-F 2 "" H 8000 5200 50  0001 C CNN
+F 1 "100n" V 7862 5200 50  0000 C CNN
+F 2 "Capacitors_SMD:C_0603_HandSoldering" H 8000 5200 50  0001 C CNN
 F 3 "~" H 8000 5200 50  0001 C CNN
 	1    8000 5200
@@
 F 0 "C304" V 7821 2900 50  0000 C CNN
 F 1 "C_Small" V 7912 2900 50  0000 C CNN
-F 2 "" H 8050 2900 50  0001 C CNN
+F 2 "Capacitors_SMD:C_0603_HandSoldering" H 8050 2900 50  0001 C CNN
 F 3 "~" H 8050 2900 50  0001 C CNN
 	1    8050 2900
@@
 F 0 "C301" H 2858 1304 50  0000 R CNN
 F 1 "100n" H 2858 1395 50  0000 R CNN
-F 2 "" H 2950 1350 50  0001 C CNN
+F 2 "Capacitors_SMD:C_0603" H 2950 1350 50  0001 C CNN
 F 3 "~" H 2950 1350 50  0001 C CNN
 	1    2950 1350
@@
 F 0 "C302" H 4518 1396 50  0000 L CNN
 F 1 "2u2" H 4518 1305 50  0000 L CNN
-F 2 "" H 4438 1200 50  0001 C CNN
+F 2 "Capacitors_SMD:C_0805" H 4438 1200 50  0001 C CNN
 F 3 "~" H 4400 1350 50  0001 C CNN
 	1    4400 1350

Commit message: Layout started, schematic modified for easier layout
Parts:
- J301, J302: footprint Connectors_Phoenix:PhoenixContact_MCV-G_02x3.81mm_Vertical -> PCBDecals:2Pin_4mm
- U301: footprint Package_TO_SOT_THT:TO-220-3_Vertical -> digikey-footprints:TO-220-3
- U302, U304: footprint Sensor_Current:Allegro_CB_PSF -> PCBDecals:Allegro_PFF
- U303, U305: footprint Package_TO_SOT_SMD:SOT-23-5 -> TO_SOT_Packages_SMD:SOT-23-5_HandSoldering
Connections:
- net labels added: ESC1_C_Negative, ESC2_C_Negative
Changed lines of the file:
@@
 F 0 "U302" H 6800 2350 50  0000 L CNN
 F 1 "ACS770xCB-100U-PSF" H 6800 1850 50  0000 L CNN
-F 2 "Sensor_Current:Allegro_CB_PSF" H 6750 2100 50  0001 C CNN
+F 2 "PCBDecals:Allegro_PFF" H 6750 2100 50  0001 C CNN
 F 3 "http://www.allegromicro.com/~/media/Files/Datasheets/ACS758-Datasheet.ashx?la=en" H 6750 2100 50  0001 C CNN
 	1    6750 2100
@@
 F 0 "U304" H 6700 4600 50  0000 L CNN
 F 1 "ACS770xCB-100U-PSF" H 6700 4100 50  0000 L CNN
-F 2 "Sensor_Current:Allegro_CB_PSF" H 6650 4350 50  0001 C CNN
+F 2 "PCBDecals:Allegro_PFF" H 6650 4350 50  0001 C CNN
 F 3 "http://www.allegromicro.com/~/media/Files/Datasheets/ACS758-Datasheet.ashx?la=en" H 6650 4350 50  0001 C CNN
 	1    6650 4350
@@
 F 0 "J301" H 7180 2742 50  0000 L CNN
 F 1 "Conn_01x02" H 7180 2651 50  0000 L CNN
-F 2 "Connectors_Phoenix:PhoenixContact_MCV-G_02x3.81mm_Vertical" H 7100 2750 50  0001 C CNN
+F 2 "PCBDecals:2Pin_4mm" H 7100 2750 50  0001 C CNN
 F 3 "~" H 7100 2750 50  0001 C CNN
 	1    7100 2750
@@
 F 0 "J302" H 7180 5042 50  0000 L CNN
 F 1 "Conn_01x02" H 7180 4951 50  0000 L CNN
-F 2 "Connectors_Phoenix:PhoenixContact_MCV-G_02x3.81mm_Vertical" H 7100 5050 50  0001 C CNN
+F 2 "PCBDecals:2Pin_4mm" H 7100 5050 50  0001 C CNN
 F 3 "~" H 7100 5050 50  0001 C CNN
 	1    7100 5050
@@
 F 0 "U305" H 7850 5700 50  0000 L CNN
 F 1 "OP179GRT" H 7850 5400 50  0000 L CNN
-F 2 "Package_TO_SOT_SMD:SOT-23-5" H 7850 5550 50  0001 C CNN
+F 2 "TO_SOT_Packages_SMD:SOT-23-5_HandSoldering" H 7850 5550 50  0001 C CNN
 F 3 "http://www.analog.com/media/en/technical-documentation/data-sheets/OP179_279.pdf" H 7850 5750 50  0001 C CNN
 	1    7850 5550
@@
 F 0 "U303" H 7950 3400 50  0000 L CNN
 F 1 "OP179GRT" H 7950 3100 50  0000 L CNN
-F 2 "Package_TO_SOT_SMD:SOT-23-5" H 7950 3250 50  0001 C CNN
+F 2 "TO_SOT_Packages_SMD:SOT-23-5_HandSoldering" H 7950 3250 50  0001 C CNN
 F 3 "http://www.analog.com/media/en/technical-documentation/data-sheets/OP179_279.pdf" H 7950 3450 50  0001 C CNN
 	1    7950 3250
@@
 F 0 "U301" H 3700 1392 50  0000 C CNN
 F 1 "LF50_TO220" H 3700 1301 50  0000 C CNN
-F 2 "Package_TO_SOT_THT:TO-220-3_Vertical" H 3700 1375 50  0001 C CIN
+F 2 "digikey-footprints:TO-220-3" H 3700 1375 50  0001 C CIN
 F 3 "http://www.st.com/content/ccc/resource/technical/document/datasheet/c4/0e/7e/2a/be/bc/4c/bd/CD00000546.pdf/files/CD00000546.pdf/jcr:content/translations/en.CD00000546.pdf" H 3700 1100 50  0001 C CNN
 	1    3700 1150
@@
 	1    0    0    -1
 $EndComp
+Text Label 6300 2700 1    50   ~ 0
+ESC1_C_Negative
+Text Label 6200 5000 1    50   ~ 0
+ESC2_C_Negative
 $EndSCHEMATC

Commit message: Layout improvements
Signed-off-by: findersee <aki.kuusela@findersee.fi>
Parts:
- removed C302: 2u2, Capacitors_SMD:C_0805, symbol Device:CP
- removed C305, C308: 100n, Capacitors_SMD:C_0603_HandSoldering, symbol Device:C_Small
- removed U301: LF50_TO220, digikey-footprints:TO-220-3, symbol Regulator_Linear:LF50_TO220
- added C302: 10n, Capacitors_SMD:C_0603_HandSoldering, symbol Device:C_Small
- added C309: 2u2, Capacitors_SMD:C_0805, symbol Device:C_Small
- added R305, R307: 12k, Resistors_SMD:R_0603_HandSoldering, symbol Device:R_Small
- added R306, R308: 18k, Resistors_SMD:R_0603_HandSoldering, symbol Device:R_Small
- added U301: LP2985-5.0, TO_SOT_Packages_SMD:SOT-23-5_HandSoldering, symbol Regulator_Linear:LP2985-5.0
- C301: value 100n -> 1u
Connections:
- wire segments 86 -> 91
Changed lines of the file:
@@
 Wire Wire Line
 	6650 3100 6650 3150
-Wire Wire Line
-	6650 3400 6650 3450
-$Comp
-L Device:C_Small C305
-U 1 1 5CE3E1F3
-P 6850 3300
-F 0 "C305" H 6758 3254 50  0000 R CNN
-F 1 "100n" H 6758 3345 50  0000 R CNN
-F 2 "Capacitors_SMD:C_0603_HandSoldering" H 6850 3300 50  0001 C CNN
-F 3 "~" H 6850 3300 50  0001 C CNN
-	1    6850 3300
-	-1   0    0    1
-$EndComp
-Wire Wire Line
-	6650 3450 6850 3450
-Wire Wire Line
-	6850 3450 6850 3400
-Connection ~ 6650 3450
-Wire Wire Line
-	6650 3450 6650 3500
-Wire Wire Line
-	6850 3200 6850 3150
 Connection ~ 6650 3150
 Wire Wire Line
 	6650 3150 6650 3200
-Connection ~ 6850 3150
 $Comp
 L Device:R_Small R303
@@
 Wire Wire Line
 	6650 5400 6650 5450
-Wire Wire Line
-	6650 5700 6650 5750
-$Comp
-L Device:C_Small C308
-U 1 1 5CE3EF03
-P 6850 5600
-F 0 "C308" H 6758 5554 50  0000 R CNN
-F 1 "100n" H 6758 5645 50  0000 R CNN
-F 2 "Capacitors_SMD:C_0603_HandSoldering" H 6850 5600 50  0001 C CNN
-F 3 "~" H 6850 5600 50  0001 C CNN
-	1    6850 5600
-	-1   0    0    1
-$EndComp
-Wire Wire Line
-	6650 5750 6850 5750
-Wire Wire Line
-	6850 5750 6850 5700
-Connection ~ 6650 5750
-Wire Wire Line
-	6650 5750 6650 5800
-Wire Wire Line
-	6850 5500 6850 5450
-Wire Wire Line
-	6850 5450 6650 5450
 Connection ~ 6650 5450
 Wire Wire Line
 	6650 5450 6650 5500
-Connection ~ 6850 5450
 Wire Wire Line
 	6200 5050 6200 4450
@@
 Wire Wire Line
 	6300 2750 6650 2750
-Wire Wire Line
-	6850 3150 6650 3150
 Wire Wire Line
 	6200 5050 6650 5050
@@
 Text GLabel 8400 3250 2    50   Output ~ 0
 ESC1_VOLTAGE_OUT
-Text GLabel 7200 4350 2    50   Output ~ 0
+Text GLabel 8400 4350 2    50   Output ~ 0
 ESC2_CURRENT_OUT
-Text GLabel 7250 2100 2    50   Output ~ 0
+Text GLabel 8400 2100 2    50   Output ~ 0
 ESC1_CURRENT_OUT
-Wire Wire Line
-	7250 2100 7150 2100
-Wire Wire Line
-	7200 4350 7050 4350
 $Comp
 L Device:C_Small C303
@@
 $EndComp
 Wire Wire Line
-	6850 5450 7550 5450
-Wire Wire Line
 	7550 5650 7500 5650
 Wire Wire Line
@@
 Wire Wire Line
 	8150 5200 8150 5250
-Wire Wire Line
-	6850 3150 7650 3150
 $Comp
 L power:GND #PWR0311
@@
 Wire Wire Line
 	8350 3250 8250 3250
-$Comp
-L Regulator_Linear:LF50_TO220 U301
-U 1 1 5CEB32A3
-P 3700 1150
-F 0 "U301" H 3700 1392 50  0000 C CNN
-F 1 "LF50_TO220" H 3700 1301 50  0000 C CNN
-F 2 "digikey-footprints:TO-220-3" H 3700 1375 50  0001 C CIN
-F 3 "http://www.st.com/content/ccc/resource/technical/document/datasheet/c4/0e/7e/2a/be/bc/4c/bd/CD00000546.pdf/files/CD00000546.pdf/jcr:content/translations/en.CD00000546.pdf" H 3700 1100 50  0001 C CNN
-	1    3700 1150
-	1    0    0    -1
-$EndComp
-$Comp
-L Device:C_Small C301
-U 1 1 5CEB3613
-P 2950 1350
-F 0 "C301" H 2858 1304 50  0000 R CNN
-F 1 "100n" H 2858 1395 50  0000 R CNN
-F 2 "Capacitors_SMD:C_0603" H 2950 1350 50  0001 C CNN
-F 3 "~" H 2950 1350 50  0001 C CNN
-	1    2950 1350
-	-1   0    0    1
-$EndComp
-$Comp
-L Device:CP C302
-U 1 1 5CEB371B
-P 4400 1350
-F 0 "C302" H 4518 1396 50  0000 L CNN
-F 1 "2u2" H 4518 1305 50  0000 L CNN
-F 2 "Capacitors_SMD:C_0805" H 4438 1200 50  0001 C CNN
-F 3 "~" H 4400 1350 50  0001 C CNN
-	1    4400 1350
-	1    0    0    -1
-$EndComp
-Wire Wire Line
-	4400 1200 4400 1150
-Wire Wire Line
-	4400 1150 4000 1150
-Wire Wire Line
-	2950 1250 2950 1150
-Wire Wire Line
-	2950 1150 3400 1150
-Wire Wire Line
-	2950 1150 2600 1150
-Connection ~ 2950 1150
-Wire Wire Line
-	3700 1450 3700 1550
-Wire Wire Line
-	3700 1550 4400 1550
-Wire Wire Line
-	4400 1550 4400 1500
+Wire Wire Line
+	2950 1250 2950 1050
+Wire Wire Line
+	2950 1050 2600 1050
+Wire Wire Line
+	3700 1550 4250 1550
 Wire Wire Line
 	3700 1550 2950 1550
@@
 Wire Wire Line
 	3700 1600 3700 1550
-Text GLabel 4650 1150 2    50   Output ~ 0
+Text GLabel 4850 1050 2    50   Output ~ 0
 +5VA
 Wire Wire Line
-	4650 1150 4400 1150
-Connection ~ 4400 1150
+	4850 1050 4600 1050
 $Comp
 L power:VCC #PWR0301
 U 1 1 5CEBEF98
-P 2600 1150
-F 0 "#PWR0301" H 2600 1000 50  0001 C CNN
-F 1 "VCC" H 2617 1323 50  0000 C CNN
-F 2 "" H 2600 1150 50  0001 C CNN
-F 3 "" H 2600 1150 50  0001 C CNN
-	1    2600 1150
+P 2600 1050
+F 0 "#PWR0301" H 2600 900 50  0001 C CNN
+F 1 "VCC" H 2617 1223 50  0000 C CNN
+F 2 "" H 2600 1050 50  0001 C CNN
+F 3 "" H 2600 1050 50  0001 C CNN
+	1    2600 1050
 	1    0    0    -1
 $EndComp
@@
 Text Label 6200 5000 1    50   ~ 0
 ESC2_C_Negative
+$Comp
+L Device:R_Small R305
+U 1 1 5CEA144F
+P 7800 2100
+F 0 "R305" V 7604 2100 50  0000 C CNN
+F 1 "12k" V 7700 2100 50  0000 C CNN
+F 2 "Resistors_SMD:R_0603_HandSoldering" H 7800 2100 50  0001 C CNN
+F 3 "~" H 7800 2100 50  0001 C CNN
+	1    7800 2100
+	0    1    1    0
+$EndComp
+$Comp
+L Device:R_Small R306
+U 1 1 5CEA1520
+P 7950 2250
+F 0 "R306" H 8009 2296 50  0000 L CNN
+F 1 "18k" H 8009 2205 50  0000 L CNN
+F 2 "Resistors_SMD:R_0603_HandSoldering" H 7950 2250 50  0001 C CNN
+F 3 "~" H 7950 2250 50  0001 C CNN
+	1    7950 2250
+	-1   0    0    -1
+$EndComp
+$Comp
+L power:GND #PWR0320
+U 1 1 5CEA15B7
+P 7950 2400
+F 0 "#PWR0320" H 7950 2150 50  0001 C CNN
+F 1 "GND" H 7955 2227 50  0000 C CNN
+F 2 "" H 7950 2400 50  0001 C CNN
+F 3 "" H 7950 2400 50  0001 C CNN
+	1    7950 2400
+	1    0    0    -1
+$EndComp
+Wire Wire Line
+	7150 2100 7700 2100
+Wire Wire Line
+	7900 2100 7950 2100
+Wire Wire Line
+	7950 2100 7950 2150
+Connection ~ 7950 2100
+Wire Wire Line
+	7950 2100 8400 2100
+Wire Wire Line
+	7950 2350 7950 2400
+$Comp
+L Device:R_Small R307
+U 1 1 5CEA9170
+P 7800 4350
+F 0 "R307" V 7604 4350 50  0000 C CNN
+F 1 "12k" V 7700 4350 50  0000 C CNN
+F 2 "Resistors_SMD:R_0603_HandSoldering" H 7800 4350 50  0001 C CNN
+F 3 "~" H 7800 4350 50  0001 C CNN
+	1    7800 4350
+	0    1    1    0
+$EndComp
+$Comp
+L Device:R_Small R308
+U 1 1 5CEA9176
+P 7950 4500
+F 0 "R308" H 8009 4546 50  0000 L CNN
+F 1 "18k" H 8009 4455 50  0000 L CNN
+F 2 "Resistors_SMD:R_0603_HandSoldering" H 7950 4500 50  0001 C CNN
+F 3 "~" H 7950 4500 50  0001 C CNN
+	1    7950 4500
+	-1   0    0    -1
+$EndComp
+$Comp
+L power:GND #PWR0321
+U 1 1 5CEA917C
+P 7950 4650
+F 0 "#PWR0321" H 7950 4400 50  0001 C CNN
+F 1 "GND" H 7955 4477 50  0000 C CNN
+F 2 "" H 7950 4650 50  0001 C CNN
+F 3 "" H 7950 4650 50  0001 C CNN
+	1    7950 4650
+	1    0    0    -1
+$EndComp
+Wire Wire Line
+	7900 4350 7950 4350
+Wire Wire Line
+	7950 4350 7950 4400
+Connection ~ 7950 4350
+Wire Wire Line
+	7950 4350 8400 4350
+Wire Wire Line
+	7950 4600 7950 4650
+Wire Wire Line
+	7050 4350 7700 4350
+$Comp
+L Regulator_Linear:LP2985-5.0 U301
+U 1 1 5CEB555D
+P 3700 1150
+F 0 "U301" H 3700 1492 50  0000 C CNN
+F 1 "LP2985-5.0" H 3700 1401 50  0000 C CNN
+F 2 "TO_SOT_Packages_SMD:SOT-23-5_HandSoldering" H 3700 1475 50  0001 C CNN
+F 3 "http://www.ti.com/lit/ds/symlink/lp2985.pdf" H 3700 1150 50  0001 C CNN
+	1    3700 1150
+	1    0    0    -1
+$EndComp
+Wire Wire Line
+	4100 1050 4600 1050
+Connection ~ 4600 1050
+$Comp
+L Device:C_Small C302
+U 1 1 5CEBF878
+P 4250 1350
+F 0 "C302" H 4342 1396 50  0000 L CNN
+F 1 "10n" H 4342 1305 50  0000 L CNN
+F 2 "Capacitors_SMD:C_0603_HandSoldering" H 4250 1350 50  0001 C CNN
+F 3 "~" H 4250 1350 50  0001 C CNN
+	1    4250 1350
+	1    0    0    -1
+$EndComp
+Wire Wire Line
+	4100 1150 4250 1150
+Wire Wire Line
+	4250 1150 4250 1250
+Wire Wire Line
+	4250 1450 4250 1550
+Connection ~ 4250 1550
+Wire Wire Line
+	4250 1550 4600 1550
+Wire Wire Line
+	3300 1050 3150 1050
+Connection ~ 2950 1050
+Wire Wire Line
+	3300 1150 3150 1150
+Wire Wire Line
+	3150 1150 3150 1050
+Connection ~ 3150 1050
+Wire Wire Line
+	3150 1050 2950 1050
+$Comp
+L Device:C_Small C301
+U 1 1 5CEB3613
+P 2950 1350
+F 0 "C301" H 2858 1304 50  0000 R CNN
+F 1 "1u" H 2858 1395 50  0000 R CNN
+F 2 "Capacitors_SMD:C_0603" H 2950 1350 50  0001 C CNN
+F 3 "~" H 2950 1350 50  0001 C CNN
+	1    2950 1350
+	-1   0    0    1
+$EndComp
+$Comp
+L Device:C_Small C309
+U 1 1 5CEC8EFA
+P 4600 1350
+F 0 "C309" H 4508 1304 50  0000 R CNN
+F 1 "2u2" H 4508 1395 50  0000 R CNN
+F 2 "Capacitors_SMD:C_0805" H 4600 1350 50  0001 C CNN
+F 3 "~" H 4600 1350 50  0001 C CNN
+	1    4600 1350
+	-1   0    0    1
+$EndComp
+Wire Wire Line
+	4600 1050 4600 1250
+Wire Wire Line
+	4600 1450 4600 1550
+Wire Wire Line
+	3700 1450 3700 1550
+Wire Wire Line
+	6650 5700 6650 5800
+Wire Wire Line
+	6650 5450 7550 5450
+Wire Wire Line
+	6650 3150 7650 3150
+Wire Wire Line
+	6650 3400 6650 3500
 $EndSCHEMATC

Commit message: Added SWD connector for debugging
Parts:
- removed U303, U305: OP179GRT, TO_SOT_Packages_SMD:SOT-23-5_HandSoldering, symbol Amplifier_Operational:OP179GRT
- added U303, U305: MCP6001-OT, Package_TO_SOT_SMD:SOT-23-5, symbol Amplifier_Operational:MCP6001-OT
Changed lines of the file:
@@
 	6650 4000 6650 4050
-$Comp
-L Amplifier_Operational:OP179GRT U305
-U 1 1 5CE5D469
-P 7850 5550
-F 0 "U305" H 7850 5700 50  0000 L CNN
-F 1 "OP179GRT" H 7850 5400 50  0000 L CNN
-F 2 "TO_SOT_Packages_SMD:SOT-23-5_HandSoldering" H 7850 5550 50  0001 C CNN
-F 3 "http://www.analog.com/media/en/technical-documentation/data-sheets/OP179_279.pdf" H 7850 5750 50  0001 C CNN
-	1    7850 5550
-	1    0    0    -1
-$EndComp
-$Comp
-L Amplifier_Operational:OP179GRT U303
-U 1 1 5CE5D4E3
-P 7950 3250
-F 0 "U303" H 7950 3400 50  0000 L CNN
-F 1 "OP179GRT" H 7950 3100 50  0000 L CNN
-F 2 "TO_SOT_Packages_SMD:SOT-23-5_HandSoldering" H 7950 3250 50  0001 C CNN
-F 3 "http://www.analog.com/media/en/technical-documentation/data-sheets/OP179_279.pdf" H 7950 3450 50  0001 C CNN
-	1    7950 3250
-	1    0    0    -1
-$EndComp
 $Comp
 L power:+5VA #PWR0307
@@
 Wire Wire Line
 	6650 3400 6650 3500
+$Comp
+L Amplifier_Operational:MCP6001-OT U303
+U 1 1 5CEC3C95
+P 7950 3250
+F 0 "U303" H 7950 3450 50  0000 L CNN
+F 1 "MCP6001-OT" H 7950 3050 50  0001 L CNN
+F 2 "Package_TO_SOT_SMD:SOT-23-5" H 7850 3050 50  0001 L CNN
+F 3 "http://ww1.microchip.com/downloads/en/DeviceDoc/21733j.pdf" H 7950 3450 50  0001 C CNN
+	1    7950 3250
+	1    0    0    -1
+$EndComp
+$Comp
+L Amplifier_Operational:MCP6001-OT U305
+U 1 1 5CEC3EEF
+P 7850 5550
+F 0 "U305" H 7850 5750 50  0000 L CNN
+F 1 "MCP6001-OT" H 7850 5350 50  0001 L CNN
+F 2 "Package_TO_SOT_SMD:SOT-23-5" H 7750 5350 50  0001 L CNN
+F 3 "http://ww1.microchip.com/downloads/en/DeviceDoc/21733j.pdf" H 7850 5750 50  0001 C CNN
+	1    7850 5550
+	1    0    0    -1
+$EndComp
 $EndSCHEMATC

Commit message: Changed the digital potentiometer to AD5160 10k version and enabled SPI3
Parts:
- U303, U305: footprint Package_TO_SOT_SMD:SOT-23-5 -> TO_SOT_Packages_SMD:SOT-23-5_HandSoldering
Changed lines of the file:
@@
 F 0 "U303" H 7950 3450 50  0000 L CNN
 F 1 "MCP6001-OT" H 7950 3050 50  0001 L CNN
-F 2 "Package_TO_SOT_SMD:SOT-23-5" H 7850 3050 50  0001 L CNN
+F 2 "TO_SOT_Packages_SMD:SOT-23-5_HandSoldering" H 7850 3050 50  0001 L CNN
 F 3 "http://ww1.microchip.com/downloads/en/DeviceDoc/21733j.pdf" H 7950 3450 50  0001 C CNN
 	1    7950 3250
@@
 F 0 "U305" H 7850 5750 50  0000 L CNN
 F 1 "MCP6001-OT" H 7850 5350 50  0001 L CNN
-F 2 "Package_TO_SOT_SMD:SOT-23-5" H 7750 5350 50  0001 L CNN
+F 2 "TO_SOT_Packages_SMD:SOT-23-5_HandSoldering" H 7750 5350 50  0001 L CNN
 F 3 "http://ww1.microchip.com/downloads/en/DeviceDoc/21733j.pdf" H 7850 5750 50  0001 C CNN
 	1    7850 5550

Commit message: Added cooling temperature sensor
Parts:
- C304: value C_Small -> 100n
Changed lines of the file:
@@
 P 8050 2900
 F 0 "C304" V 7821 2900 50  0000 C CNN
-F 1 "C_Small" V 7912 2900 50  0000 C CNN
+F 1 "100n" V 7912 2900 50  0000 C CNN
 F 2 "Capacitors_SMD:C_0603_HandSoldering" H 8050 2900 50  0001 C CNN
 F 3 "~" H 8050 2900 50  0001 C CNN
