File: hw/Telemetry.kicad_pcb (KiCad board)
At the start: 4 copper layers, 100 x 82 mm, 130 parts, among them J101 BOOT0, J102 BOOT0, J103 SPORT, J104 SBUS, J105 USB_B_Micro, J106 UART_EXP, J201 Conn_01x02, J301 Conn_01x02, J302 Conn_01x02, J401 Conn_01x02, J402 Conn_01x02, J403 Conn_01x02, J404 Conn_01x02, J405 Conn_01x02, J406 Conn_01x02, J407 Conn_01x02, J408 Conn_01x02, J409 SERVO_OUT, J410 AUDIO, Q201 AO3401A, Q202 AO3401A, Q203 IRLML6344TRPBF, Q204 IRLML6344TRPBF, Q401 IRLML6344TRPBF, Q402 IRLML6344TRPBF, Q403 IRLML6344TRPBF, Q404 CSD17306Q5A, Q405 IRLML6344TRPBF, Q406 IRLML6344TRPBF, Q407 IRLML6344TRPBF, Q408 CSD17306Q5A, SW101 SW_Push, U101 STM32F303CBx, U102 IS25LP032D, U201 AP1501-K5, U202 RT6200, U301 LP2985-5.0, U302 ACS770xCB-100U-PSF, U303 MCP6001-OT, U304 ACS770xCB-100U-PSF, U305 MCP6001-OT, U401 MCP1416, U402 MCP1416, U403 AD5160BRJZ10-R2, U404 MCP6001-OT, X101 SG-310_SCF_8.000000MHZ

Commit message: Layout and gerber update
Routing:
- net GND: vias 86 -> 93
- net /Current measurement/ESC2_C_Negative: vias 0 -> 7
- net /Current measurement/ESC1_C_Negative: vias 0 -> 7
- net +BATT: vias 4 -> 22
- added copper zone on VCC, net +3V3
- added copper zone on VCC, net +BATT
- added copper zone on VCC, net /Current measurement/ESC1_C_Negative
- added copper zone on VCC, net /Current measurement/ESC2_C_Negative
- added copper zone on GND, net GND
- added copper zone on VCC, net VCC
- removed copper zone on In2.Cu, net +3V3
- removed copper zone on In2.Cu, net +BATT
- removed copper zone on In2.Cu, net /Current measurement/ESC1_C_Negative
- removed copper zone on In2.Cu, net /Current measurement/ESC2_C_Negative
- removed copper zone on In1.Cu, net GND
- removed copper zone on In2.Cu, net VCC
Changed lines of the file:
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@@
     (thickness 1.6)
     (drawings 7)
-    (tracks 1166)
+    (tracks 1209)
     (zones 0)
     (modules 130)
@@
   (layers
     (0 F.Cu signal)
-    (1 In1.Cu signal)
-    (2 In2.Cu signal)
+    (1 GND power)
+    (2 VCC power)
     (31 B.Cu signal)
     (32 B.Adhes user)
@@
     (47 F.CrtYd user)
     (48 B.Fab user)
-    (49 F.Fab user hide)
+    (49 F.Fab user)
   )
   (setup
@@
       (viasonmask true)
       (mode 1)
-      (useauxorigin true)
+      (useauxorigin false)
       (hpglpennumber 1)
       (hpglpenspeed 20)
@@
   (segment (start 126 92.07) (end 125.82 92.25) (width 0.25) (layer F.Cu) (net 1))
   (segment (start 125.82 92.25) (end 125.82 93.74) (width 0.25) (layer F.Cu) (net 1))
+  (via (at 105.9 70.2) (size 1.2) (drill 0.6) (layers F.Cu B.Cu) (net 1))
+  (via (at 105.9 74.4) (size 1.2) (drill 0.6) (layers F.Cu B.Cu) (net 1))
+  (via (at 105.9 78.5) (size 1.2) (drill 0.6) (layers F.Cu B.Cu) (net 1))
+  (via (at 105.9 77.1) (size 1.2) (drill 0.6) (layers F.Cu B.Cu) (net 1))
+  (via (at 105.9 75.8) (size 1.2) (drill 0.6) (layers F.Cu B.Cu) (net 1))
+  (via (at 105.9 73) (size 1.2) (drill 0.6) (layers F.Cu B.Cu) (net 1))
+  (via (at 105.9 71.6) (size 1.2) (drill 0.6) (layers F.Cu B.Cu) (net 1))
   (segment (start 137.5 62.7) (end 136.9 62.1) (width 0.25) (layer F.Cu) (net 2))
   (segment (start 138.35 62.7) (end 137.5 62.7) (width 0.25) (layer F.Cu) (net 2) (status 10))
@@
   (segment (start 153 46) (end 151 44) (width 0.25) (layer F.Cu) (net 2))
   (segment (start 154.2 46) (end 153 46) (width 0.25) (layer F.Cu) (net 2))
-  (segment (start 71.25 74.45) (end 69.95 73.15) (width 0.25) (layer F.Cu) (net 3) (status 10))
+  (via (at 92.4 58.5) (size 1.2) (drill 0.6) (layers F.Cu B.Cu) (net 3))
+  (segment (start 71.25 74.45) (end 70.4 73.6) (width 0.25) (layer F.Cu) (net 3) (status 10))
   (segment (start 71.4 74.45) (end 71.25 74.45) (width 0.25) (layer F.Cu) (net 3) (status 30))
-  (segment (start 69.95 73.15) (end 69.95 71.35) (width 0.25) (layer F.Cu) (net 3))
-  (segment (start 68.499999 70.000001) (end 65 73.5) (width 0.25) (layer F.Cu) (net 3) (status 20))
+  (segment (start 69.95 73.15) (end 69.95 71.6) (width 0.25) (layer F.Cu) (net 3))
+  (segment (start 68.499999 70.000001) (end 68.499999 70.000001) (width 0.25) (layer F.Cu) (net 3) (status 20))
   (segment (start 68.600001 70.000001) (end 68.499999 70.000001) (width 0.25) (layer F.Cu) (net 3))
   (segment (start 69.95 71.35) (end 68.600001 70.000001) (width 0.25) (layer F.Cu) (net 3))
@@
   (segment (start 76.5 82.3) (end 77.7 82.3) (width 0.6) (layer F.Cu) (net 3))
   (segment (start 74.2 80) (end 76.5 82.3) (width 0.6) (layer F.Cu) (net 3))
-  (segment (start 65 73.5) (end 71.5 80) (width 0.6) (layer F.Cu) (net 3))
+  (segment (start 65 73.5) (end 68.5 77) (width 0.6) (layer F.Cu) (net 3))
   (segment (start 71.5 80) (end 74.2 80) (width 0.6) (layer F.Cu) (net 3))
   (segment (start 76.55 98.3) (end 76.5 98.35) (width 0.6) (layer F.Cu) (net 3))
@@
   (segment (start 111.9 106.35) (end 112.8 105.45) (width 0.6) (layer F.Cu) (net 3))
   (segment (start 125.2 105.15) (end 123.4 105.15) (width 0.6) (layer F.Cu) (net 3))
+  (via (at 69.6 62.5) (size 1.2) (drill 0.6) (layers F.Cu B.Cu) (net 3))
+  (via (at 69.6 61) (size 1.2) (drill 0.6) (layers F.Cu B.Cu) (net 3))
+  (via (at 69.6 59.4) (size 1.2) (drill 0.6) (layers F.Cu B.Cu) (net 3))
+  (via (at 69.6 64) (size 1.2) (drill 0.6) (layers F.Cu B.Cu) (net 3))
+  (via (at 68.6 58) (size 1.2) (drill 0.6) (layers F.Cu B.Cu) (net 3))
+  (via (at 69.6 65.5) (size 1.2) (drill 0.6) (layers F.Cu B.Cu) (net 3))
+  (via (at 68.5 66.9) (size 1.2) (drill 0.6) (layers F.Cu B.Cu) (net 3))
+  (via (at 92.4 62.4) (size 1.2) (drill 0.6) (layers F.Cu B.Cu) (net 3))
+  (via (at 92.4 61.1) (size 1.2) (drill 0.6) (layers F.Cu B.Cu) (net 3))
+  (via (at 92.4 59.8) (size 1.2) (drill 0.6) (layers F.Cu B.Cu) (net 3))
+  (via (at 92.4 63.7) (size 1.2) (drill 0.6) (layers F.Cu B.Cu) (net 3))
+  (via (at 92.4 65) (size 1.2) (drill 0.6) (layers F.Cu B.Cu) (net 3))
+  (segment (start 68.499999 70.000001) (end 65 73.5) (width 0.25) (layer F.Cu) (net 3) (status 20))
+  (via (at 68.499999 70.000001) (size 1.2) (drill 0.6) (layers F.Cu B.Cu) (net 3))
+  (segment (start 68.5 77) (end 71.5 80) (width 0.6) (layer F.Cu) (net 3))
+  (via (at 68.5 77) (size 1.2) (drill 0.6) (layers F.Cu B.Cu) (net 3))
+  (segment (start 70.4 73.6) (end 69.95 73.15) (width 0.25) (layer F.Cu) (net 3) (status 10))
+  (via (at 70.4 73.6) (size 1.2) (drill 0.6) (layers F.Cu B.Cu) (net 3))
+  (segment (start 69.95 71.6) (end 69.95 71.35) (width 0.25) (layer F.Cu) (net 3))
+  (via (at 69.95 71.6) (size 1.2) (drill 0.6) (layers F.Cu B.Cu) (net 3))
+  (via (at 69.8 75.5) (size 1.2) (drill 0.6) (layers F.Cu B.Cu) (net 3))
   (segment (start 114.1 79.75) (end 114 79.65) (width 0.6) (layer F.Cu) (net 4))
   (segment (start 115.1 79.75) (end 114.1 79.75) (width 0.6) (layer F.Cu) (net 4) (status 10))
@@
   (segment (start 129.75 68.4) (end 129.85 68.3) (width 0.25) (layer F.Cu) (net 21))
   (segment (start 129.75 69.35) (end 129.75 68.4) (width 0.25) (layer F.Cu) (net 21) (status 10))
+  (via (at 65.2 45.4) (size 1.2) (drill 0.6) (layers F.Cu B.Cu) (net 22))
+  (via (at 66.7 45.5) (size 1.2) (drill 0.6) (layers F.Cu B.Cu) (net 22))
+  (via (at 63.7 45.5) (size 1.2) (drill 0.6) (layers F.Cu B.Cu) (net 22))
   (segment (start 77.35 41.65) (end 73 46) (width 0.3) (layer F.Cu) (net 22) (status 20))
   (segment (start 87.95 41.65) (end 87.1 41.65) (width 0.3) (layer F.Cu) (net 22) (status 10))
   (segment (start 87.5 41.65) (end 87.1 41.65) (width 0.3) (layer F.Cu) (net 22) (status 10))
   (segment (start 87.1 41.65) (end 77.35 41.65) (width 0.3) (layer F.Cu) (net 22))
+  (via (at 69.4 51.4) (size 1.2) (drill 0.6) (layers F.Cu B.Cu) (net 22))
+  (via (at 69.4 52.8) (size 1.2) (drill 0.6) (layers F.Cu B.Cu) (net 22))
+  (via (at 69.4 54.2) (size 1.2) (drill 0.6) (layers F.Cu B.Cu) (net 22))
+  (via (at 69.4 50) (size 1.2) (drill 0.6) (layers F.Cu B.Cu) (net 22))
+  (via (at 101.3 52.3) (size 1.2) (drill 0.6) (layers F.Cu B.Cu) (net 23))
+  (via (at 101.3 49.5) (size 1.2) (drill 0.6) (layers F.Cu B.Cu) (net 23))
+  (via (at 101.3 53.7) (size 1.2) (drill 0.6) (layers F.Cu B.Cu) (net 23))
+  (via (at 101.3 50.9) (size 1.2) (drill 0.6) (layers F.Cu B.Cu) (net 23))
   (segment (start 109.6 41.4) (end 105 46) (width 0.3) (layer F.Cu) (net 23) (status 20))
   (segment (start 120.3 41.4) (end 119.3 41.4) (width 0.25) (layer F.Cu) (net 23))
   (segment (start 119.85 41.4) (end 119.3 41.4) (width 0.3) (layer F.Cu) (net 23))
   (segment (start 119.3 41.4) (end 109.6 41.4) (width 0.3) (layer F.Cu) (net 23))
+  (via (at 95.7 45.5) (size 1.2) (drill 0.6) (layers F.Cu B.Cu) (net 23))
+  (via (at 98.7 45.5) (size 1.2) (drill 0.6) (layers F.Cu B.Cu) (net 23))
+  (via (at 97.2 45.4) (size 1.2) (drill 0.6) (layers F.Cu B.Cu) (net 23))
   (segment (start 145.51 74.04) (end 145.5 74.05) (width 1) (layer F.Cu) (net 24) (status 30))
   (segment (start 148.45 74.04) (end 145.51 74.04) (width 1) (layer F.Cu) (net 24) (status 30))
@@
     )
   )
-  (zone (net 1) (net_name GND) (layer In1.Cu) (hatch edge 0.508)
+  (zone (net 1) (net_name GND) (layer GND) (hatch edge 0.508)
     (connect_pads (clearance 0.3))
     (min_thickness 0.22)
@@
     )
   )
-  (zone (net 4) (net_name VCC) (layer In2.Cu) (hatch edge 0.508)
+  (zone (net 4) (net_name VCC) (layer VCC) (hatch edge 0.508)
     (connect_pads (clearance 0.4))
     (min_thickness 0.22)
@@
     )
   )
-  (zone (net 2) (net_name +3V3) (layer In2.Cu) (hatch edge 0.508)
+  (zone (net 2) (net_name +3V3) (layer VCC) (hatch edge 0.508)
     (priority 1)
     (connect_pads (clearance 0.3))
@@
     )
   )
-  (zone (net 23) (net_name "/Current measurement/ESC2_C_Negative") (layer In2.Cu) (hatch edge 0.508)
+  (zone (net 23) (net_name "/Current measurement/ESC2_C_Negative") (layer VCC) (hatch edge 0.508)
     (priority 1)
     (connect_pads (clearance 0.3))
@@
     )
   )
-  (zone (net 22) (net_name "/Current measurement/ESC1_C_Negative") (layer In2.Cu) (hatch edge 0.508)
+  (zone (net 22) (net_name "/Current measurement/ESC1_C_Negative") (layer VCC) (hatch edge 0.508)
     (priority 1)
     (connect_pads (clearance 0.3))
@@
     )
   )
-  (zone (net 3) (net_name +BATT) (layer In2.Cu) (hatch edge 0.508)
+  (zone (net 3) (net_name +BATT) (layer VCC) (hatch edge 0.508)
     (priority 2)
     (connect_pads (clearance 0.3))
@@
     )
   )
-  (zone (net 0) (net_name "") (layers In1.Cu B.Cu) (hatch edge 0.508)
+  (zone (net 0) (net_name "") (layers GND B.Cu) (hatch edge 0.508)
     (connect_pads (clearance 0.4))
     (min_thickness 0.254)
@@
     )
   )
-  (zone (net 0) (net_name "") (layers In1.Cu B.Cu) (hatch edge 0.508)
+  (zone (net 0) (net_name "") (layers GND B.Cu) (hatch edge 0.508)
     (connect_pads (clearance 0.4))
     (min_thickness 0.254)
